File: hardware/projects/OBC_PCB/OBC_PCB.kicad_sch (KiCad schematic)
At the start: 0 parts

Commit message: Adding most basic components to schematic
Parts:
- added ANT1: SGGP.12.4.A.02, obc:SGGP124A02, symbol obc:SGGP.12.4.A.02
- added J1: 503566-2102, obc:5035662102, symbol obc:503566-2102
- added J2: DM3CS-SF, obc:HRS_DM3CS-SF, symbol obc:DM3CS-SF
- added J3: USB4720-03-A, obc:GCT_USB4720-03-A_REVA, symbol obc:USB4720-03-A
- added U1: MAX-M10S, RF_GPS:ublox_MAX, symbol RF_GPS:MAX-M10S
- added U2: NPM1300-CAAA-R, obc:BGA35N44X41P5X7_237X307X51, symbol obc:NPM1300-CAAA-R
- added U3: BMA400, obc:QFN_BMA400_BOS, symbol obc:BMA400
- added U4: BMM350, obc:BGA9_BMM350, symbol obc:BMM350
- added U5: BMP581, obc:BMP581, symbol obc:BMP581
- added U6: nRF54LM20A-PAXX, obc:Nordic_FCCSP-98_3.67x3.85mm_Layout10x10_P0.35mm_Offcenter, symbol obc:nRF54LM20A-PAXX
Connections:
- new net: U1.1 (GND), U1.10 (GND), U1.12 (GND)
- new net: U6.A1 (VSS), U6.A10 (VSS), U6.A7 (VSS), U6.D1 (VSS), U6.D2 (VSS), U6.E5 (VSS), U6.E6 (VSS), U6.F1 (VSS), U6.F5 (VSS), U6.F6 (VSS), U6.K1 (VSS), U6.K10 (VSS)
- new net: U6.A3 (VDD), U6.A4 (VDD), U6.A9 (VDD), U6.G10 (VDD), U6.H1 (VDD)
Other:
- added sheet Power Management (..\..\shared\power_management.kicad_sch)

Commit message: more kicad work
Parts:
- removed J3: USB4720-03-A, obc:GCT_USB4720-03-A_REVA, symbol obc:USB4720-03-A
- removed U2: NPM1300-CAAA-R, obc:BGA35N44X41P5X7_237X307X51, symbol obc:NPM1300-CAAA-R
- added ANT2: 2450AT18B100, RF_Antenna:Johanson_2450AT18x100, symbol Device:Antenna_Chip
- added C20: 4.7uF, Capacitor_SMD:C_0603_1608Metric, symbol Device:C
- added C21, C40: 10uF, Capacitor_SMD:C_0603_1608Metric, symbol Device:C
- added C22, C23, C24, C33, C34, C35, C37, C39, C41, C43, C44, C45, C46, C47, C48: 100nF, Capacitor_SMD:C_0402_1005Metric, symbol Device:C
- added C25: 4.7uF, Capacitor_SMD:C_0402_1005Metric, symbol Device:C
- added C26, C28, C42: 2.2uF, Capacitor_SMD:C_0402_1005Metric, symbol Device:C
- added C27: 1.0pF, symbol Device:C
- added C29: 1.2pF, Capacitor_SMD:C_0402_1005Metric, symbol Device:C
- added C30: 1.5pF, Capacitor_SMD:C_0402_1005Metric, symbol Device:C
- added C31: DNP, Capacitor_SMD:C_0402_1005Metric, symbol Device:C
- added C32, C36, C38: 1uF, Capacitor_SMD:C_0402_1005Metric, symbol Device:C
- added D3: GREEN, LED_SMD:LED_0603_1608Metric, symbol Device:LED
- added FB1: 120R@100MHz, Inductor_SMD:L_0402_1005Metric, symbol Device:FerriteBead
- added J5: SWD, Connector_PinHeader_1.27mm:PinHeader_2x05_P1.27mm_Vertical_SMD, symbol Connector:Conn_ARM_JTAG_SWD_10
- added L10: 3.6nH, Inductor_SMD:L_0402_1005Metric, symbol Device:L
- added L11: 4.7nH, Inductor_SMD:L_0402_1005Metric, symbol Device:L
- added L12: 3.3nH, Inductor_SMD:L_0402_1005Metric, symbol Device:L
- added L4: 4.7uH, Inductor_SMD:L_0603_1608Metric, symbol Device:L
- added L6: 1.0nH, Inductor_SMD:L_0402_1005Metric, symbol Device:L
- added R10, R11, R12, R13, R14: 47k, Resistor_SMD:R_0402_1005Metric, symbol Device:R
- added R20: 10k, Resistor_SMD:R_0402_1005Metric, symbol Device:R
- added R21, R22, R23, R24: 4.7k, Resistor_SMD:R_0402_1005Metric, symbol Device:R
- added R4: 200R 1%, Resistor_SMD:R_0402_1005Metric, symbol Device:R
- added R5: 2.2R, Resistor_SMD:R_0402_1005Metric, symbol Device:R
- added R8: 1k, Resistor_SMD:R_0402_1005Metric, symbol Device:R
- added R9: 33R, Resistor_SMD:R_0402_1005Metric, symbol Device:R
- added SW1: PREV, Button_Switch_SMD:SW_SPST_EVQP7C, symbol Switch:SW_Push
- added SW2: NEXT, Button_Switch_SMD:SW_SPST_EVQP7C, symbol Switch:SW_Push
- added SW3: SELECT, Button_Switch_SMD:SW_SPST_EVQP7C, symbol Switch:SW_Push
- added SW4: BACK, Button_Switch_SMD:SW_SPST_EVQP7C, symbol Switch:SW_Push
- added TP1: GPS_SAFEBOOT, TestPoint:TestPoint_Pad_D1.5mm, symbol Connector:TestPoint
- added TP2: DBG_TX, TestPoint:TestPoint_Pad_D1.5mm, symbol Connector:TestPoint
- added TP3: DBG_RX, TestPoint:TestPoint_Pad_D1.5mm, symbol Connector:TestPoint
- added Y1: 32MHz 8pF, Crystal:Crystal_SMD_2016-4Pin_2.0x1.6mm, symbol Device:Crystal_GND24
- added Y2: 32.768kHz 9pF, Crystal:Crystal_SMD_2012-2Pin_2.0x1.2mm, symbol Device:Crystal
Connections:
- net at ANT1.1 (RF_FEED): now also U1.11 (RF_IN)
- net GND: now reaches ANT1.2 (GND)
- net GND: now also ANT1.3 (GND), ANT1.4 (GND), ANT1.5 (GND), ANT1.6 (GND), ANT1.7 (GND), ANT1.8 (GND), ANT1.9 (GND), J1.10, J1.MP1, J1.MP2, J2.6 (VSS), J2.S1 (GND), J2.S2 (GND), J2.S3 (GND), J2.S5 (GND), U1.1 (GND), U1.10 (GND), U1.12 (GND), U3.1 (SDO), U3.8 (GNDIO), U3.9 (GND), U4.B1 (GND), U4.C3 (BYPASS), U5.3 (VSS), U5.8 (VSS), U5.9 (VSS), U6.A1 (VSS), U6.A10 (VSS), U6.A7 (VSS), U6.D1 (VSS), U6.D2 (VSS), U6.E5 (VSS), U6.E6 (VSS), U6.F1 (VSS), U6.F5 (VSS), U6.F6 (VSS), U6.K1 (VSS), U6.K10 (VSS), C20.2, C21.2, C22.2, C23.2, C24.2, C25.2, C26.2, C28.2, C29.2, C30.2, C31.2, C32.2, C33.2, C34.2, C35.2, C36.2, C37.2, C38.2, C39.2, C40.2, C41.2, C42.2, C43.2, C44.2, C45.2, C46.2, C47.2, C48.2, D3.1 (K), J5.3 (GND), J5.5 (GND), J5.9 (GNDDetect), R4.1, SW1.2, SW2.2, SW3.2, SW4.2, Y1.2 (G), Y1.4 (G)
- net GPS_SDA: now reaches U1.16 (SDA)
- net GPS_SDA: now also U6.J8 (P1.06), R21.2
- net GPS_SCL: now reaches U1.17 (SCL)
- net GPS_SCL: now also U6.G8 (P1.07), R22.2
- net GPS_SAFEBOOT: now reaches U1.18 (~{SAFEBOOT})
- net GPS_SAFEBOOT: now also TP1.1
- net GPS_TXD: now reaches U1.2 (TXD)
- net GPS_TXD: now also U6.J2 (P0.03)
- net GPS_RXD: now reaches U1.3 (RXD)
- net GPS_RXD: now also U6.E3 (P0.09)
- net GPS_TIMEPULSE: now reaches U1.4 (TIMEPULSE)
- net GPS_TIMEPULSE: now also U6.J9 (P1.04)
- net GPS_EXTINT: now reaches U1.5 (EXTINT)
- net GPS_EXTINT: now also U6.H8 (P1.05)
- net +3V3: now reaches U1.6 (V_BCKP)
- net +3V3: now also J1.9, U3.10 (CSB), U3.3 (VDDIO), U3.7 (VDD), U4.B2 (ADSEL), U4.B3 (VDDIO), U5.1 (VDDIO), U5.10 (VDD), U5.5 (SDO), U5.6 (CSB), U6.A3 (VDD), U6.A4 (VDD), U6.A9 (VDD), U6.G10 (VDD), U6.H1 (VDD), C21.1, C22.1, C23.1, C24.1, C35.1, C38.1, C39.1, C43.1, C44.1, C45.1, C46.1, C47.1, J5.1 (VTref), R20.1, R23.1, R24.1
- net +3V3_GPS: now reaches U1.7 (VCC_IO)
- net +3V3_GPS: now also U1.8 (VCC), C32.1, C33.1, C34.1, R21.1, R22.1
- net DISP_R0: now reaches U6.B10 (P2.00)
- net DISP_R0: now also J1.13
- net SD_SCK: now reaches U6.B9 (P2.06)
- net SD_SCK: now also R9.1
- net DISP_R1: now reaches U6.C10 (P2.01)
- net DISP_R1: now also J1.14
- net DISP_BCK: now reaches U6.C9 (P2.07)
- net DISP_BCK: now also J1.12
- net DISP_G0: now reaches U6.D10 (P2.02)
- net DISP_G0: now also J1.15
- net SD_MOSI: now reaches U6.D9 (P2.08)
- net SD_MOSI: now also J2.3 (CMD), R10.2
- net DISP_G1: now reaches U6.E10 (P2.03)
- net DISP_G1: now also J1.16
- net SD_MISO: now reaches U6.E9 (P2.09)
- net SD_MISO: now also J2.7 (DAT0), R11.2
- net DISP_B0: now reaches U6.F10 (P2.04)
- net DISP_B0: now also J1.17
- net SD_CS: now reaches U6.F9 (P2.10)
- net SD_CS: now also J2.2 (CD/DAT3), R12.2
- net DISP_B1: now reaches U6.G9 (P2.05)
- net DISP_B1: now also J1.18
- net +5V_DISP: now reaches J1.1
- net +5V_DISP: now also C36.1, C37.1
- net DISP_BSP: now reaches J1.11
- net DISP_BSP: now also U6.G5 (P3.07)
- net DISP_VCOM: now reaches J1.20
- net DISP_VCOM: now also U6.H7 (P3.00)
- net DISP_GSP: now reaches J1.3
- net DISP_GSP: now also U6.H4 (P3.03)
- net DISP_GCK: now reaches J1.4
- net DISP_GCK: now also U6.J4 (P3.04)
- net DISP_GEN: now reaches J1.5
- net DISP_GEN: now also U6.G7 (P3.05)
- net DISP_INTB: now reaches J1.6
- net DISP_INTB: now also U6.G6 (P3.06)
- net DISP_VB: now reaches J1.7
- net DISP_VB: now also U6.H6 (P3.01)
- net DISP_VA: now reaches J1.8
- net DISP_VA: now also U6.H5 (P3.02)
- net PMIC_INT: now reaches U6.F3 (P0.08)
- net BTN_BACK: now reaches U6.G3 (P0.07)
- net BTN_BACK: now also SW4.1
- net BTN_NEXT: now reaches U6.H2 (P0.06)
- net BTN_NEXT: now also SW2.1
- net BTN_PREV: now reaches U6.H3 (P0.05)
- net BTN_PREV: now also SW1.1
- net BTN_SELECT: now reaches U6.J1 (P0.04)
- net BTN_SELECT: now also SW3.1
- net SCL: now reaches U6.J3 (P0.02)
- net SCL: now also U3.12 (SCX), U4.A3 (SCK), U5.2 (SCK), R24.2
- net SDA: now reaches U6.K2 (P0.01)
- net SDA: now also U3.2 (SDX), U4.A2 (SDA), U5.4 (SDI), R23.2
- net ACC_INT1: now reaches U6.K3 (P0.00)
- net ACC_INT1: now also U3.5 (INT1)
- net BARO_INT: now reaches U5.7 (INT)
- net BARO_INT: now also U6.K8 (P1.00)
- net LED_DBG: now reaches U6.F4 (P3.10)
- net LED_DBG: now also R8.1
- net DISP_5V_EN: now reaches U6.F7 (P3.09)
- net SD_CD: now reaches U6.G4 (P3.08)
- net SD_CD: now also J2.9 (CD_SW)
- net at U6.A2 (XC1): now also Y1.3
- net DCC: now reaches U6.A5 (DCC)
- net DCC: now also L4.1
- net DECD: now reaches U6.A6 (DECD)
- net DECD: now also C25.1, FB1.1, L4.2
- net DECA: now reaches U6.A8 (DECA)
- net DECA: now also C26.1, C27.1, FB1.2, L6.1
- net at U6.B1 (XC2): now also Y1.1
- net DECRF: now reaches U6.C1 (DECRF)
- net DECRF: now also C27.2, L6.2
- net at U6.C6 (P1.20): now also Y2.1
- net at U6.C7 (P1.21): now also Y2.2
- net at U6.E1 (ANT): now also L10.1
- net nRESET: now reaches U6.F2 (~{RESET})
- net nRESET: now also J5.10 (~{RESET}), R20.2
- net SWDCLK: now reaches U6.G1 (SWDCLK)
- net SWDCLK: now also J5.4 (SWCLK/TCK)
- net SWDIO: now reaches U6.G2 (SWDIO)
- net SWDIO: now also J5.2 (SWDIO/TMS)
- net at U6.J5 (TXRTUNE): now also R4.2
- net USB_DM: now reaches U6.K4 (D-)
- net USB_DP: now reaches U6.K5 (D+)
- net at U6.K6 (DECUSB): now also C28.1
- net at U6.K7 (VBUS): now also C20.1, R5.2
- net MAG_INT: now reaches U4.A1 (INT)
- net MAG_INT: now also U6.H9 (P1.03)
- net +1V8_MAG: now reaches U4.C1 (VDD)
- net +1V8_MAG: now also C48.1
- net at U4.C2 (CRST): now also C42.1
- net SD_DAT2: now reaches J2.1 (DAT2)
- net SD_DAT2: now also R14.2
- net +3V3_SD: now reaches J2.4 (VDD)
- net +3V3_SD: now also C40.1, C41.1, R10.1, R11.1, R12.1, R13.1, R14.1
- net at J2.5 (CLK): now also R9.2
- net SD_DAT1: now reaches J2.8 (DAT1)
- net SD_DAT1: now also R13.2
- net DBG_RX: now reaches U6.E8 (P1.09)
- net DBG_RX: now also TP3.1
- net DBG_TX: now reaches U6.F8 (P1.08)
- net DBG_TX: now also TP2.1
- new net: D3.2 (A), R8.2
- new net: C30.1, L11.2, L12.1
- new net: ANT2.1 (FEED), C31.1, L12.2
- new net: C29.1, L10.2, L11.1
- new net VBUS_MCU: R5.1
- no-connect marks 0 -> 38
Other:
- note added: "50R, keep short"
- note added: "BMA400"
- note added: "BMM350 (VDD on 1V8)"
- note added: "BMP581"
- note added: "BUTTONS (to GND, internal pull-ups, fw debounce)"
- note added: "CRST: 2.2uF non-magnetic, right at ball"
- note added: "DEBUG — SWD + UART TP"
- note added: "DISPLAY — LS021B7DD02 (21p FPC)"
- note added: "GPS — MAX-M10S + PATCH"
- note added: "NOTES Shared I2C (TWIM30, P0.01/P0.02, pulls 4.7k -> +3V3): nPM1300 0x6B / BMP581 0x47 / BMA400 0x14 / BMM350 0x15 GPS I2C (TWIM2x, P1.06/P1.07): MAX-M10S 0x42, pulls -> +3V3_GPS (gated rail, no backfeed when GPS is off) SD card: SPIM00 fast SPI 16/32 MHz - SCK P2.06 / MOSI P2.08 / MISO P2.09 / CS P2.10 (Nordic-mandated SPIM00 pins; set P2 extra-high drive E0/E1 for 32 MHz). Rail +3V3_SD = BUCK1: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"
- note added: "P0 (wake / I2C / buttons) P1 (GPS / debug)"
- note added: "P2 (fast: display bus + SD SPI) P3 (COM / gate / misc)"
- note added: "POWER"
- note added: "SENSORS — shared I2C: BMP581 0x47 / BMA400 0x14 / BMM350 0x15"
- note added: "USB-C input, Li-Ion charger, BUCK1 (+3V3_SD), BUCK2 (+3V3), LDO 1.8V (mag), GPS load switch, 5V display boost -> page 2"
- note added: "VDD1 (3V3)"
- note added: "VDD2 (5V gate)"
- note added: "at VDD balls"
- note added: "internal load caps - no ext. CL"
- note added: "microSD — DM3CS-SF (SPI mode)"
- note added: "nRF54LM20A — SYSTEM / RF / USB"
- note added: "pulls to +3V3_SD (gated) - no backfeed when SD off"
- company: (none) -> OpenBikeComputer
- title: (none) -> OpenBikeComputer — main board
- moved on the sheet: ANT1, J1, J2, U1, U3, U4, U5, U6A, U6B, U6C, U6D, U6E

Commit message: more pcb work - add baseboard remove Proto
Other:
- sheet Power Management: file ..\..\shared\power_management.kicad_sch -> ../../shared/power_management.kicad_sch
- sheet Power Management ports: added USB_DM, USB_DP; removed none

Commit message: Add Fit_Test PCB and work on Schematic
Parts:
- removed C36, C38: 1uF, Capacitor_SMD:C_0402_1005Metric, symbol Device:C
- removed C37, C39, C41: 100nF, Capacitor_SMD:C_0402_1005Metric, symbol Device:C
- removed C40: 10uF, Capacitor_SMD:C_0603_1608Metric, symbol Device:C
- removed D3: GREEN, LED_SMD:LED_0603_1608Metric, symbol Device:LED
- removed J1: 503566-2102, obc:5035662102, symbol obc:503566-2102
- removed R10, R11, R12, R13, R14: 47k, Resistor_SMD:R_0402_1005Metric, symbol Device:R
- removed R8: 1k, Resistor_SMD:R_0402_1005Metric, symbol Device:R
- added J1: LS021B7DD02, obc:5035662102, symbol obc:LS021B7DD02
Connections:
- net SD_DAT1 is gone; now on net DISP.R1: J2.8 (DAT1)
- net SD_DAT2 is gone; now on net SD_Card.DAT2: J2.1 (DAT2)
- net +3V3: now also J1.9 (VDD1)
- net +5V_DISP: now also J1.1 (VDD2)
- net BARO_INT: no longer U6.K8 (P1.00)
- net DBG_RX: no longer U6.E8 (P1.09)
- net DBG_TX: no longer U6.F8 (P1.08)
- net GND: now also J1.10 (VSS)
- net GPS_EXTINT: no longer U6.H8 (P1.05)
- net GPS_SCL: no longer U6.G8 (P1.07)
- net GPS_SDA: no longer U6.J8 (P1.06)
- net GPS_TIMEPULSE: no longer U6.J9 (P1.04)
- net MAG_INT: no longer U6.H9 (P1.03)
- net SD_Card.CLK: now reaches J2.5 (CLK), R9.2
- net DISP.VCOM: now reaches U6.B2 (P1.15)
- net DISP.VCOM: now also J1.20 (VCOM)
- net DISP.VB: now reaches U6.B3 (P1.16)
- net DISP.VB: now also J1.7 (VB)
- net DISP.VA: now reaches U6.B4 (P1.17)
- net DISP.VA: now also J1.8 (VA)
- net DISP.BSP: now reaches U6.C2 (P1.14)
- net DISP.BSP: now also J1.11 (BSP)
- net DISP.INTB: now reaches U6.C3 (P1.13)
- net DISP.INTB: now also J1.6 (INTB)
- net DISP.GEN: now reaches U6.C4 (P1.12)
- net DISP.GEN: now also J1.5 (GEN)
- net DISP.GCK: now reaches U6.C5 (P1.11)
- net DISP.GCK: now also J1.4 (GCK)
- net DISP.GSP: now reaches U6.D5 (P1.10)
- net DISP.GSP: now also J1.3 (GSP)
- net DISP_B0 renamed DISP.R1
- net DISP.R1: now also J1.14 (R1)
- net DISP_B1 renamed SD_Card.CMD
- net SD_Card.CMD: now also J2.3 (CMD)
- net DISP_BCK renamed DISP.BCK
- net DISP.BCK: now also J1.12 (BCK)
- net DISP_BSP: no longer names the net of U6.G5 (P3.07)
- net DISP_G0 renamed SD_Card.DAT0
- net SD_Card.DAT0: now also J2.7 (DAT0)
- net DISP_G1 renamed SD_Card.DAT2
- net DISP_GCK: no longer names the net of U6.J4 (P3.04)
- net DISP_GEN: no longer names the net of U6.G7 (P3.05)
- net DISP_GSP: no longer names the net of U6.H4 (P3.03)
- net DISP_INTB: no longer names the net of U6.G6 (P3.06)
- net DISP_R0 renamed DISP.R0
- net DISP.R0: now also J2.2 (CD/DAT3), J1.13 (R0)
- net DISP_R1: no longer names the net of U6.C10 (P2.01)
- net DISP_R1: now also R9.1
- net DISP_VA: no longer names the net of U6.H5 (P3.02)
- net DISP_VB: no longer names the net of U6.H6 (P3.01)
- net DISP_VCOM: no longer names the net of U6.H7 (P3.00)
- net LED_DBG: no longer names the net of U6.F4 (P3.10)
- net SD_CD: no longer names the net of U6.G4 (P3.08)
- net SD_CD: no longer J2.9 (CD_SW)
- net SD_CS renamed DISP.B1
- net DISP.B1: now also J1.18 (B1); no longer J2.2 (CD/DAT3)
- net SD_MISO renamed DISP.B0
- net DISP.B0: now also J1.17 (B0); no longer J2.7 (DAT0)
- net SD_MOSI renamed DISP.G1
- net DISP.G1: now also J1.16 (G1); no longer J2.3 (CMD)
- net SD_SCK renamed DISP.G0
- net DISP.G0: now also J1.15 (G0); no longer R9.1
- new net: J1.19 (NC), J1.2 (NC), J1.21 (NC), J1.MP1, J1.MP2
- no-connect marks 38 -> 12
Other:
- note removed: "NOTES Shared I2C (TWIM30, P0.01/P0.02, pulls 4.7k -> +3V3): nPM1300 0x6B / BMP581 0x47 / BMA400 0x14 / BMM350 0x15 GPS I2C (TWIM2x, P1.06/P1.07): MAX-M10S 0x42, pulls -> +3V3_GPS (gated rail, no backfeed when GPS is off) SD card: SPIM00 fast SPI 16/32 MHz - SCK P2.06 / MOSI P2.08 / MISO P2.09 / CS P2.10 (Nordic-mandated SPIM00 pins; set P2 extra-high drive E0/E1 for 32 MHz). Rail +3V3_SD = BUCK1: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"
- note removed: "P0 (wake / I2C / buttons) P1 (GPS / debug)"
- note removed: "P2 (fast: display bus + SD SPI) P3 (COM / gate / misc)"
- note removed: "VDD1 (3V3)"
- note removed: "VDD2 (5V gate)"
- note removed: "pulls to +3V3_SD (gated) - no backfeed when SD off"
- moved on the sheet: C42, C43, C44, C45, C46, C47, C48, J2, R23, R24, R9, U3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

Commit message: more schematic progress and some library additions
Parts:
- removed ANT2: 2450AT18B100, RF_Antenna:Johanson_2450AT18x100, symbol Device:Antenna_Chip
- removed C20: 4.7uF, Capacitor_SMD:C_0603_1608Metric, symbol Device:C
- removed C21: 10uF, Capacitor_SMD:C_0603_1608Metric, symbol Device:C
- removed C22, C23, C24, C33, C34, C35, C43, C44, C45, C46, C47, C48: 100nF, Capacitor_SMD:C_0402_1005Metric, symbol Device:C
- removed C25: 4.7uF, Capacitor_SMD:C_0402_1005Metric, symbol Device:C
- removed C26, C28: 2.2uF, Capacitor_SMD:C_0402_1005Metric, symbol Device:C
- removed C27: 1.0pF, symbol Device:C
- removed C29: 1.2pF, Capacitor_SMD:C_0402_1005Metric, symbol Device:C
- removed C30: 1.5pF, Capacitor_SMD:C_0402_1005Metric, symbol Device:C
- removed C31: DNP, Capacitor_SMD:C_0402_1005Metric, symbol Device:C
- removed C32: 1uF, Capacitor_SMD:C_0402_1005Metric, symbol Device:C
- removed FB1: 120R@100MHz, Inductor_SMD:L_0402_1005Metric, symbol Device:FerriteBead
- removed L10: 3.6nH, Inductor_SMD:L_0402_1005Metric, symbol Device:L
- removed L11: 4.7nH, Inductor_SMD:L_0402_1005Metric, symbol Device:L
- removed L12: 3.3nH, Inductor_SMD:L_0402_1005Metric, symbol Device:L
- removed L4: 4.7uH, Inductor_SMD:L_0603_1608Metric, symbol Device:L
- removed L6: 1.0nH, Inductor_SMD:L_0402_1005Metric, symbol Device:L
- removed R5: 2.2R, Resistor_SMD:R_0402_1005Metric, symbol Device:R
- removed TP1: GPS_SAFEBOOT, TestPoint:TestPoint_Pad_D1.5mm, symbol Connector:TestPoint
- removed TP2: DBG_TX, TestPoint:TestPoint_Pad_D1.5mm, symbol Connector:TestPoint
- removed TP3: DBG_RX, TestPoint:TestPoint_Pad_D1.5mm, symbol Connector:TestPoint
- removed Y1: 32MHz 8pF, Crystal:Crystal_SMD_2016-4Pin_2.0x1.6mm, symbol Device:Crystal_GND24
- removed Y2: 32.768kHz 9pF, Crystal:Crystal_SMD_2012-2Pin_2.0x1.2mm, symbol Device:Crystal
- added C11: 2.2u, symbol Device:C_Small
- added C12: 4.7u, symbol Device:C_Small
- added C13: 1p, symbol Device:C_Small
- added L3: 4.7uH, symbol Device:L_Small
- added L4: L_Ferrite_Small, symbol Device:L_Ferrite_Small
- added L6: 1.0nH, symbol Device:L_Small
- added Y1: 32MHz 8pF, symbol Device:Crystal_Small
- added Y3: 32.768kHz 9pF, symbol Device:Crystal_Small
- SW1, SW2, SW3: footprint Button_Switch_SMD:SW_SPST_EVQP7C -> obc:TL1016AAF220QG
Connections:
- net USB_DM is gone; now on net Power Management/USB_DP: U6.K4 (D-)
- net USB_DP is gone; now on net Power Management/USB_DM: U6.K5 (D+)
- net GND: now also C11.2, C12.2
- net SWDCLK: no longer U6.G1 (SWDCLK)
- net SWDIO: no longer U6.G2 (SWDIO)
- net nRESET: no longer U6.F2 (~{RESET})
- net at U6.K6 (DECUSB): now also C11.1
- net at U6.B1 (XC2): now also Y1.1
- net at U6.A2 (XC1): now also Y1.2
- net at U6.C6 (P1.20): now also Y3.2
- net at U6.C7 (P1.21): now also Y3.1
- net DCC: no longer names the net of U6.A5 (DCC)
- net DCC: now also L3.1
- net DECA: no longer names the net of U6.A8 (DECA)
- net DECA: now also C13.1, L4.2, L6.2
- net DECD: no longer names the net of U6.A6 (DECD)
- net DECD: now also C12.1, L3.2, L4.1
- net DECRF: no longer names the net of U6.C1 (DECRF)
- net DECRF: now also C13.2, L6.1
Other:
- note removed: "BMA400"
- note removed: "BMM350 (VDD on 1V8)"
- note removed: "BMP581"
- note removed: "at VDD balls"
- note removed: "internal load caps - no ext. CL"
- moved on the sheet: U6A

Commit message: hardware: complete modular main-board and USB schematics
Parts:
- removed ANT1: SGGP.12.4.A.02, obc:SGGP124A02, symbol obc:SGGP.12.4.A.02
- removed C42: 2.2uF, Capacitor_SMD:C_0402_1005Metric, symbol Device:C
- removed J1: LS021B7DD02, obc:5035662102, symbol obc:LS021B7DD02
- removed J2: DM3CS-SF, obc:HRS_DM3CS-SF, symbol obc:DM3CS-SF
- removed R21, R22, R23, R24: 4.7k, Resistor_SMD:R_0402_1005Metric, symbol Device:R
- removed U1: MAX-M10S, RF_GPS:ublox_MAX, symbol RF_GPS:MAX-M10S
- removed U3: BMA400, obc:QFN_BMA400_BOS, symbol obc:BMA400
- removed U4: BMM350, obc:BGA9_BMM350, symbol obc:BMM350
- removed U5: BMP581, obc:BMP581, symbol obc:BMP581
- added BZ1: CPT-9019A-SMT-TR, obc:CPT-9019A-SMT-TR, symbol obc:CPT-9019A-SMT-TR
- added C21: 10u, Capacitor_SMD:C_0402_1005Metric, symbol Device:C_Small
- added C22, C23, C24: 100n, Capacitor_SMD:C_0402_1005Metric, symbol Device:C_Small
- added C25: 2.2u, Capacitor_SMD:C_0201_0603Metric, symbol Device:C_Small
- added C26: 4.7u, Capacitor_SMD:C_0402_1005Metric, symbol Device:C_Small
- added C44: 1u, Capacitor_SMD:C_0402_1005Metric, symbol Device:C_Small
- added R33: 1k, Resistor_SMD:R_0402_1005Metric, symbol Device:R_Small
- added R34: 100k, Resistor_SMD:R_0402_1005Metric, symbol Device:R_Small
- added R5: 2.2R, Resistor_SMD:R_0402_1005Metric, symbol Device:R_Small
- added TP10: +5V_DISP, TestPoint:TestPoint_Pad_D1.0mm, symbol Connector:TestPoint
- added TP11: SCL, TestPoint:TestPoint_Pad_D1.0mm, symbol Connector:TestPoint
- added TP12: SDA, TestPoint:TestPoint_Pad_D1.0mm, symbol Connector:TestPoint
- added TP3: VBAT, TestPoint:TestPoint_Pad_D1.0mm, symbol Connector:TestPoint
- added TP4: VSYS, TestPoint:TestPoint_Pad_D1.0mm, symbol Connector:TestPoint
- added TP5: +3V2, TestPoint:TestPoint_Pad_D1.0mm, symbol Connector:TestPoint
- added TP6: GND, TestPoint:TestPoint_Pad_D1.0mm, symbol Connector:TestPoint
- added TP7: +3V2_GPS, TestPoint:TestPoint_Pad_D1.0mm, symbol Connector:TestPoint
- added TP8: +3V3_SD, TestPoint:TestPoint_Pad_D1.0mm, symbol Connector:TestPoint
- added TP9: +1V8_MAG, TestPoint:TestPoint_Pad_D1.0mm, symbol Connector:TestPoint
- C11: footprint (none) -> Capacitor_SMD:C_0402_1005Metric; Dielectric (none) -> X5R; Tolerance (none) -> 10%; Voltage (none) -> 10V
- C12: footprint (none) -> Capacitor_SMD:C_0201_0603Metric; Dielectric (none) -> X5R; MPN (none) -> GRM035R60J475ME15J; Manufacturer (none) -> Murata; Tolerance (none) -> 20%; Voltage (none) -> 6.3V
- C13: footprint (none) -> Capacitor_SMD:C_0201_0603Metric; Dielectric (none) -> C0G; MPN (none) -> GJM0335C1E1R0WB01D; Manufacturer (none) -> Murata; Tolerance (none) -> 0.05pF; Voltage (none) -> 25V
- J5: value SWD -> TC2030-CTX-NL; footprint Connector_PinHeader_1.27mm:PinHeader_2x05_P1.27mm_Vertical_SMD -> Connector:Tag-Connect_TC2030-IDC-NL_2x03_P1.27mm_Vertical; symbol Connector:Conn_ARM_JTAG_SWD_10 -> obc:TC2030_CTX_NL; Assembly (none) -> PCB pads only; no connector or solder paste; Cable pinout (none) -> 1 VTref, 2 SWDIO, 3 nRESET, 4 SWCLK, 5 GND, 6 SWO (unused); now left out of the parts list
- L3: footprint (none) -> Inductor_SMD:L_0603_1608Metric; DCR (none) -> 650mOhm max; MPN (none) -> MLZ1608M4R7WT000; Manufacturer (none) -> TDK; Rated Current (none) -> 350mA typ (20C rise); Saturation Current (none) -> 120mA (50% L drop); Tolerance (none) -> 20%
- L4: value L_Ferrite_Small -> 120R; footprint (none) -> Inductor_SMD:L_0201_0603Metric; DCR (none) -> 500mOhm max; Impedance frequency (none) -> 100MHz; MPN (none) -> BLM03AG121SN1D; Manufacturer (none) -> Murata; Rated Current (none) -> 200mA; Tolerance (none) -> 25%
- L6: footprint (none) -> Inductor_SMD:L_0201_0603Metric; MPN (none) -> LQP03TN1N0C02D; Manufacturer (none) -> Murata; Rated Current (none) -> 750mA; Tolerance (none) -> 0.2nH
- R20, R9: symbol Device:R -> Device:R_Small; Power (none) -> 63mW; Technology (none) -> Thick film; Tolerance (none) -> 1%; Voltage (none) -> 50V
- R4: value 200R 1% -> 200R; symbol Device:R -> Device:R_Small; Power (none) -> 63mW; Technology (none) -> Thick film; Tolerance (none) -> 1%; Voltage (none) -> 50V
- SW1, SW2: Bounce (none) -> 10ms max; Contact Material (none) -> Silver; Current Rating (none) -> 50mA; MPN (none) -> TL1016AAF220QG; Manufacturer (none) -> E-Switch; Operating Force (none) -> 220gf +80/-70gf; Operating Temperature (none) -> -40 to +85 C; Voltage Rating (none) -> 12VDC
- SW3: value SELECT -> SELECT / POWER; Bounce (none) -> 10ms max; Contact Material (none) -> Silver; Current Rating (none) -> 50mA; MPN (none) -> TL1016AAF220QG; Manufacturer (none) -> E-Switch; Operating Force (none) -> 220gf +80/-70gf; Operating Temperature (none) -> -40 to +85 C; Voltage Rating (none) -> 12VDC
- SW4: footprint Button_Switch_SMD:SW_SPST_EVQP7C -> obc:TL1016AAF220QG; Bounce (none) -> 10ms max; Contact Material (none) -> Silver; Current Rating (none) -> 50mA; MPN (none) -> TL1016AAF220QG; Manufacturer (none) -> E-Switch; Operating Force (none) -> 220gf +80/-70gf; Operating Temperature (none) -> -40 to +85 C; Voltage Rating (none) -> 12VDC
- U6: value nRF54LM20A-PAXX -> nRF54LM20A-PAAA; MPN nRF54LM20A-PAXX -> nRF54LM20A-PAAA
- Y1: value 32MHz 8pF -> 32MHz; footprint (none) -> Crystal:Crystal_SMD_2016-4Pin_2.0x1.6mm; symbol Device:Crystal_Small -> Device:Crystal_GND24_Small; Frequency tolerance (none) -> 40ppm total; Load Capacitance (none) -> 8pF; MPN (none) -> CX2016DB32000D0WZRC1; Manufacturer (none) -> Kyocera
- Y3: value 32.768kHz 9pF -> 32.768kHz; footprint (none) -> Crystal:Crystal_SMD_2012-2Pin_2.0x1.2mm; Initial tolerance (none) -> 20ppm; Load Capacitance (none) -> 9pF; MPN (none) -> 9HT11-32.768KDZC-T; Manufacturer (none) -> TXC
Connections:
- net +1V8_MAG: now also TP9.1
- net +3V3_SD: now also TP8.1
- net +5V_DISP: now also TP10.1
- net GND: now also Y1.2 (G), Y1.4 (G), BZ1.2, C21.2, C22.2, C23.2, C24.2, C25.2, C26.2, R34.2, TP6.1; no longer J5.3 (GND), J5.9 (GNDDetect)
- net SCL: now also TP11.1
- net SDA: now also TP12.1
- net SWDCLK: now also U6.G1 (SWDCLK)
- net SWDIO: now also U6.G2 (SWDIO)
- net nRESET: now also J5.3 (~{RESET}), U6.F2 (~{RESET}); no longer J5.10 (~{RESET})
- net at C13.1, L4.2, L6.2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: now also C25.1
- net at U6.D4 (P3.12): now also R33.1
- net BACKLIGHT_PWM: now reaches U6.E4 (P3.11)
- net at Y1.1: now also U6.A2 (XC1); no longer U6.B1 (XC2)
- net at Y3.1: now also U6.C6 (P1.20); no longer U6.C7 (P1.21)
- net at Y3.2: now also U6.C7 (P1.21); no longer U6.C6 (P1.20)
- net Radio/ANT: now reaches U6.E1 (ANT)
- net at U6.K7 (VBUS): now also C26.1, R5.2
- net +3V3 renamed +3V2
- net +3V2: now also C21.1, C22.1, C23.1, C24.1, TP5.1
- net BTN_SELECT: no longer names the net of U6.J1 (P0.04)
- net BTN_SELECT: no longer SW3.1
- net DISP.B0 renamed FLPR.P09
- net DISP.B1 renamed FLPR.P10
- net DISP.BCK renamed FLPR.P07
- net DISP.BSP renamed LCD.BSP
- net DISP.G0 renamed FLPR.P06
- net DISP.G1 renamed FLPR.P08
- net DISP.GCK renamed LCD.GCK
- net DISP.GEN renamed LCD.GEN
- net DISP.GSP renamed LCD.GSP
- net DISP.INTB renamed LCD.INTB
- net DISP.R0 renamed FLPR.P00
- net DISP.R1 renamed FLPR.P04
- net DISP.VA renamed LCD.VA
- net DISP.VB renamed LCD.VB
- net DISP.VCOM renamed LCD.VCOM
- net Power Management/USB_DM renamed Power Management/USB_D+
- net Power Management/USB_DP renamed Power Management/USB_D-
- net SD_Card.CLK renamed FLPR.P01
- net SD_Card.CMD renamed FLPR.P05
- net SD_Card.DAT0 renamed FLPR.P02
- net SD_Card.DAT2 renamed FLPR.P03
- new net: BZ1.1, C44.2, R34.1
- new net: C44.1, R33.2
- new net: U6.B1 (XC2), Y1.3
- new net +3V2_GPS: TP7.1
- new net Power Management/SHPHLD: SW3.1
- new net USB_VBUS: R5.1
- new net VBAT: TP3.1
- new net VSYS: TP4.1
- no-connect marks 12 -> 34
Other:
- added sheet Display (display.kicad_sch)
- added sheet GNSS (gnss.kicad_sch)
- added sheet Radio (radio.kicad_sch)
- added sheet Sensors (sensors.kicad_sch)
- added sheet Storage (storage.kicad_sch)
- sheet Power Management ports: added DISP_5V_EN, PMIC_INT, SCL, SDA, SHPHLD, USB_D+, USB_D-, USB_VBUS; removed USB_DM, USB_DP
- note added: "2.4GHz / PCB MIFA"
- note added: "BMP581 / BMA400 / BMM350"
- note added: "BUTTONS — ACTIVE LOW"
- note added: "C22 at A3/A4/A9; C23 at G10; C24 at H1. Place regulator bypass at the corresponding balls."
- note added: "Charger / 3.2V system / 3.3V SD / 1.8V MAG / GPS switch / 5V display"
- note added: "Configure HF/LF internal load caps before starting crystals. Keep crystal traces short and clear of DCC / USB."
- note added: "DEBUG — CORTEX SWD"
- note added: "Enable VREGMAIN DC/DC in firmware."
- note added: "LS021B7DD02 display"
- note added: "MAX-F11N L1/L5 GNSS"
- note added: "Native 4-bit microSD"
- note added: "P2.00: LCD R0 / SD DAT3 P2.04: LCD R1 / SD DAT1 Intentional FLPR time-sharing."
- note added: "PIEZO — 4kHz"
- note added: "POWER PROBE PADS"
- note added: "PREV/NEXT/BACK: GPIO pull-ups; firmware debounce. SELECT: PMIC_INT + SHPHLDSTATUS; enable SHPHLD events. Hold SELECT 10s: hardware power cycle (PMIC default)."
- note added: "PWM: H0H1 drive, 50% duty; idle low. C44 blocks DC. Keep acoustic port clear. Verify audibility in the sealed enclosure."
- note added: "R9: place at U6; tune from CLK waveform."
- note added: "TC2030-CTX-NL: bare pads; no solder paste. VTref = +3V2 sense only. SWO unused; RTT over SWD. Keep probe access and alignment holes clear."
- note removed: "50R, keep short"
- note removed: "BUTTONS (to GND, internal pull-ups, fw debounce)"
- note removed: "CRST: 2.2uF non-magnetic, right at ball"
- note removed: "DEBUG — SWD + UART TP"
- note removed: "DISPLAY — LS021B7DD02 (21p FPC)"
- note removed: "GPS — MAX-M10S + PATCH"
- note removed: "SENSORS — shared I2C: BMP581 0x47 / BMA400 0x14 / BMM350 0x15"
- note removed: "USB-C input, Li-Ion charger, BUCK1 (+3V3_SD), BUCK2 (+3V3), LDO 1.8V (mag), GPS load switch, 5V display boost -> page 2"
- note removed: "microSD — DM3CS-SF (SPI mode)"
- moved on the sheet: C11, C12, C13, L3, L4, L6, R20, R4, U6A, Y3

Commit message: fix(hardware): apply schematic review and peripheral pin mapping
Parts:
- removed C44: 1u, Capacitor_SMD:C_0402_1005Metric, symbol Device:C_Small
- removed R34: 100k, Resistor_SMD:R_0402_1005Metric, symbol Device:R_Small
- added R41: 470R, Resistor_SMD:R_0402_1005Metric, symbol Device:R_Small
- added TP13: USB_VBUS, TestPoint:TestPoint_Pad_D1.0mm, symbol Connector:TestPoint
- C12, C13, C25: footprint Capacitor_SMD:C_0201_0603Metric -> obc:C_Nordic_0201_0603Metric
- L4, L6: footprint Inductor_SMD:L_0201_0603Metric -> obc:L_Nordic_0201_0603Metric
- R33: value 1k -> 470R; MPN (none) -> RC0402FR-07470RL; Manufacturer (none) -> Yageo
Connections:
- net BACKLIGHT_PWM: now also U6.J10 (P1.30); no longer U6.E4 (P3.11)
- net DISP_5V_EN: now also U6.H10 (P1.29); no longer U6.F7 (P3.09)
- net GND: no longer BZ1.2
- net LCD.GCK: now also U6.H8 (P1.05); no longer U6.C5 (P1.11)
- net SCL: now also U6.H9 (P1.03); no longer U6.J3 (P0.02)
- net SDA: now also U6.J9 (P1.04); no longer U6.K2 (P0.01)
- net USB_VBUS: now also TP13.1
- net at BZ1.1: now also R33.2
- net at U6.D4 (P3.12): no longer R33.1
- net PIEZO_B: now reaches U6.K8 (P1.00)
- net PIEZO_B: now also R41.1
- net PIEZO_A: now reaches U6.K9 (P1.31)
- net PIEZO_A: now also R33.1
- new net: BZ1.2, R41.2
- new net BARO_INT: U6.K2 (P0.01)
- no-connect marks 34 -> 32
Other:
- sheet Sensors ports: added BARO_INT; removed none
- note added: "LCD: R0=P2.00, R1=P2.04, G0=P2.06, G1=P2.08 B0=P2.09, B1=P2.10, BCK=P2.07. P2.00/P2.04 share SD DAT3/DAT1; FLPR arbitrates."
- note added: "PWM21 CH0/CH1: antiphase, 4kHz, 50%; 6.4Vpp. H0H1 drive; hold both pins low when silent. Keep acoustic port clear; verify enclosed audibility."
- note removed: "Charger / 3.2V system / 3.3V SD / 1.8V MAG / GPS switch / 5V display"
- note removed: "P2.00: LCD R0 / SD DAT3 P2.04: LCD R1 / SD DAT1 Intentional FLPR time-sharing."
- note removed: "POWER"
- note removed: "PWM: H0H1 drive, 50% duty; idle low. C44 blocks DC. Keep acoustic port clear. Verify audibility in the sealed enclosure."
- moved on the sheet: R33, TP11, TP12, U6B, U6C, U6E
