File: hardware/projects/OBC_PCB/OBC_PCB.kicad_sch (KiCad schematic)
At the start: 38 parts, among them J5 TC2030-CTX-NL, SW1 PREV, SW2 NEXT, SW3 SELECT / POWER, SW4 BACK, U6 nRF54LM20A-PAAA, Y1 32MHz, Y3 32.768kHz

Commit message: hardware: name critical nets and ground connector tabs
Connections:
- net SOC_DCC: now reaches L3.1, U6.A5 (DCC)
- net SOC_USB_VBUS: now reaches C26.1, R5.2, U6.K7 (VBUS)
Changed lines of the file:
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@@
 		(color 0 0 0 0)
 	)
+	(label "SOC_DCC"
+		(at 294.64 57.15 0)
+		(effects
+			(font
+				(size 1 1)
+			)
+			(justify left bottom)
+		)
+	)
+	(label "SOC_USB_VBUS"
+		(at 243.84 54.61 0)
+		(effects
+			(font
+				(size 1 1)
+			)
+			(justify left bottom)
+		)
+	)
 )
