File: hardware/projects/OBC_PCB/OBC_PCB.kicad_sch (KiCad schematic)
At the start: 38 parts, among them J5 TC2030-CTX-NL, SW1 PREV, SW2 NEXT, SW3 SELECT / POWER, SW4 BACK, U6 nRF54LM20A-PAAA, Y1 32MHz, Y3 32.768kHz

Commit message: hardware: prepare QFN schematic for non-HDI boards
Parts:
- removed BZ1: CPT-9019A-SMT-TR, obc:CPT-9019A-SMT-TR, symbol obc:CPT-9019A-SMT-TR
- removed J5: TC2030-CTX-NL, Connector:Tag-Connect_TC2030-IDC-NL_2x03_P1.27mm_Vertical, symbol obc:TC2030_CTX_NL
- removed R20: 10k, Resistor_SMD:R_0402_1005Metric, symbol Device:R_Small
- removed R33, R41: 470R, Resistor_SMD:R_0402_1005Metric, symbol Device:R_Small
- removed SW1: PREV, obc:TL1016AAF220QG, symbol Switch:SW_Push
- removed SW2: NEXT, obc:TL1016AAF220QG, symbol Switch:SW_Push
- removed SW3: SELECT / POWER, obc:TL1016AAF220QG, symbol Switch:SW_Push
- removed SW4: BACK, obc:TL1016AAF220QG, symbol Switch:SW_Push
- removed TP10: +5V_DISP, TestPoint:TestPoint_Pad_D1.0mm, symbol Connector:TestPoint
- removed TP3: VBAT, TestPoint:TestPoint_Pad_D1.0mm, symbol Connector:TestPoint
- removed TP4: VSYS, TestPoint:TestPoint_Pad_D1.0mm, symbol Connector:TestPoint
- removed TP5: +3V2, TestPoint:TestPoint_Pad_D1.0mm, symbol Connector:TestPoint
- removed TP6: GND, TestPoint:TestPoint_Pad_D1.0mm, symbol Connector:TestPoint
- removed TP7: +3V2_GPS, TestPoint:TestPoint_Pad_D1.0mm, symbol Connector:TestPoint
- removed TP8: +3V3_SD, TestPoint:TestPoint_Pad_D1.0mm, symbol Connector:TestPoint
- removed unit 5 of U6
- TP9: value +1V8_MAG -> COM_SOURCE
- U6: value nRF54LM20A-PAAA -> nRF54LM20A-QGAA; footprint obc:Nordic_FCCSP-98_3.67x3.85mm_Layout10x10_P0.35mm_Offcenter -> Package_DFN_QFN:VQFN-52-1EP_6x6mm_P0.4mm_EP4.7x4.7mm; symbol obc:nRF54LM20A-PAXX -> obc:nRF54LM20A-QGAA; License (none) -> CERN-OHL-P-2.0; hardware/libraries/LICENSE.nordic-lib-kicad; MPN nRF54LM20A-PAAA -> nRF54LM20A-QGAA-R7; Source (none) -> https://github.com/hlord2000/nordic-lib-kicad/tree/05a4dae2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
Connections:
- net +3V2: now also U6.42 (VDD), U6.51 (VDD), U6.6 (VDD); no longer U6.A3 (VDD), U6.A4 (VDD), U6.A9 (VDD), U6.G10 (VDD), U6.H1 (VDD)
- net GND: now also U6.35 (VSS), U6.45 (VSS), U6.53 (VSS); no longer U6.A1 (VSS), U6.A10 (VSS), U6.A7 (VSS), U6.D1 (VSS), U6.D2 (VSS), U6.E5 (VSS), U6.E6 (VSS), U6.F1 (VSS), U6.F5 (VSS), U6.F6 (VSS), U6.K1 (VSS), U6.K10 (VSS)
- net PMIC_INT: now also U6.29 (P0.08); no longer U6.F3 (P0.08)
- net Radio/ANT: now also U6.34 (ANT); no longer U6.E1 (ANT)
- net SCL: now also U6.13 (P1.03); no longer U6.H9 (P1.03)
- net SDA: now also U6.14 (P1.04); no longer U6.J9 (P1.04)
- net SWDCLK: now also U6.31 (SWDCLK); no longer U6.G1 (SWDCLK)
- net SWDIO: now also U6.32 (SWDIO); no longer U6.G2 (SWDIO)
- net nRESET: now also U6.33 (~{RESET}); no longer U6.F2 (~{RESET})
- net at C12.1, L3.2, L4.1: now also U6.44 (DECD); no longer U6.A6 (DECD)
- net SD_CLK_RAW: now reaches R9.1
- net SD_CLK_RAW: now also U6.1 (P2.01); no longer U6.C10 (P2.01)
- net at C13.1, C25.1, L4.2: now also L6.1, U6.46 (DECA); no longer L6.2, U6.A8 (DECA)
- net at Y1.1: now also U6.37 (XC1); no longer U6.A2 (XC1)
- net at Y1.3: now also U6.38 (XC2); no longer U6.B1 (XC2)
- net at Y3.1: now also U6.48 (P1.20); no longer U6.C6 (P1.20)
- net at Y3.2: now also U6.49 (P1.21); no longer U6.C7 (P1.21)
- net at R4.2: now also U6.21 (TXRTUNE); no longer U6.J5 (TXRTUNE)
- net at C11.1: now also U6.18 (DECUSB); no longer U6.K6 (DECUSB)
- net +1V8_MAG renamed COM_SOURCE
- net COM_SOURCE: now also U6.7 (P1.29)
- removed net ACC_INT1: U6.K3 (P0.00)
- removed net BACKLIGHT_PWM: U6.J10 (P1.30)
- removed net BARO_INT: U6.K2 (P0.01)
- removed net BTN_BACK: U6.G3 (P0.07)
- removed net BTN_NEXT: U6.H2 (P0.06)
- removed net BTN_PREV: U6.H3 (P0.05)
- removed net DISP_5V_EN: U6.H10 (P1.29)
- removed net FLPR.P00: U6.B10 (P2.00)
- net FLPR.P01 renamed Storage/SD_CLK
- removed net FLPR.P02: U6.D10 (P2.02)
- removed net FLPR.P03: U6.E10 (P2.03)
- removed net FLPR.P04: U6.F10 (P2.04)
- removed net FLPR.P05: U6.G9 (P2.05)
- removed net FLPR.P06: U6.B9 (P2.06)
- removed net FLPR.P07: U6.C9 (P2.07)
- removed net FLPR.P08: U6.D9 (P2.08)
- removed net FLPR.P09: U6.E9 (P2.09)
- removed net FLPR.P10: U6.F9 (P2.10)
- removed net GPS_RXD: U6.E3 (P0.09)
- removed net GPS_TXD: U6.J2 (P0.03)
- removed net LCD.BSP: U6.C2 (P1.14)
- removed net LCD.GCK: U6.H8 (P1.05)
- removed net LCD.GEN: U6.C4 (P1.12)
- removed net LCD.GSP: U6.D5 (P1.10)
- removed net LCD.INTB: U6.C3 (P1.13)
- removed net LCD.VA: U6.B4 (P1.17)
- removed net LCD.VB: U6.B3 (P1.16)
- removed net LCD.VCOM: U6.B2 (P1.15)
- removed net PIEZO_A: U6.K9 (P1.31)
- removed net PIEZO_B: U6.K8 (P1.00)
- removed net Power Management/USB_D+: U6.K5 (D+)
- removed net Power Management/USB_D-: U6.K4 (D-)
- net SOC_DCC: no longer names the net of L3.1
- net SOC_DCC: now also U6.43 (DCC); no longer U6.A5 (DCC)
- net SOC_USB_VBUS: no longer names the net of C26.1, R5.2
- net SOC_USB_VBUS: now also U6.17 (VBUS); no longer U6.K7 (VBUS)
- new net: C13.2, L6.2, U6.36 (DECRF)
- new net GNSS/GPS_RXD: U6.30 (P0.09)
- new net GNSS/GPS_TXD: U6.25 (P0.03)
- new net LCD_B0: U6.23 (P1.08)
- new net LCD_B1: U6.24 (P1.09)
- new net LCD_BCK: U6.15 (P1.05)
- new net LCD_BSP: U6.41 (P1.18)
- new net LCD_G0: U6.16 (P1.06)
- new net LCD_G1: U6.22 (P1.07)
- new net LCD_GCK: U6.40 (P1.16)
- new net LCD_GEN: U6.12 (P1.02)
- new net LCD_GSP: U6.11 (P1.01)
- new net LCD_INTB: U6.50 (P1.24)
- new net LCD_R0: U6.8 (P1.30)
- new net LCD_R1: U6.9 (P1.31)
- new net SD_CMD: U6.5 (P2.05)
- new net SD_D0: U6.2 (P2.02)
- new net SD_D1: U6.4 (P2.04)
- new net SD_D2: U6.3 (P2.03)
- new net SD_D3: U6.52 (P2.00)
- new net Sensors/ACC_INT1: U6.47 (P1.19)
- new net USB_D+: U6.19 (D+)
- new net USB_D-: U6.20 (D-)
- new net User I/O/BTN_BACK: U6.28 (P0.07)
- new net User I/O/BTN_NEXT: U6.27 (P0.06)
- new net User I/O/BTN_PREV: U6.26 (P0.04)
- new net User I/O/BTN_SELECT: U6.39 (P1.15)
- new net User I/O/BUZZER_PWM: U6.10 (P1.00)
- no-connect marks 32 -> 0
Other:
- added sheet User I/O (user_io.kicad_sch)
- sheet Display ports: added COM_EN, COM_SOURCE, LCD_B0, LCD_B1, LCD_BCK, LCD_BSP, LCD_G0, LCD_G1, LCD_GCK, LCD_GEN, LCD_GSP, LCD_INTB, LCD_R0, LCD_R1, SCL, SDA; removed BACKLIGHT_PWM, FLPR{P2_LINES}, LCD{LCD_CONTROL}, SHARED_R0, SHARED_R1
- sheet Power Management ports: added COM_EN, LOUD; removed DISP_5V_EN
- sheet Sensors ports: added none; removed BARO_INT
- sheet Storage ports: added SD_CLK, SD_CMD, SD_D0, SD_D1, SD_D2, SD_D3; removed FLPR{P2_LINES}, SHARED_D1, SHARED_D3
- note added: "MCU / CLOCKS / USB"
- note added: "P1.01/P1.02: disable NFC before GSP/GEN. COM: TIMER21 + GPIOTE20. ACC_INT1: P1.19 SENSE. Normal idle keeps COM and the clock screen running. Shutdown blanks the panel and removes VDD2 before VDD1."
- note added: "P2.00-05: dedicated sEMMC. R9 at MCU clock pad. The PCB retains the placement reference and needs a new layout."
- note added: "PROVISIONAL QGAA RF / REGULATOR NETWORK Obtain the Nordic LM20 QFN reference circuit. Verify matching, bypass values and geometry before fabrication."
- note added: "UARTE30: GPS_TXD is MCU RX; GPS_RXD is MCU TX. Release UART before GPS power-off. Enable LS2 before UART."
- note added: "VDD bypass: C22 at pad 6; C23 at pad 42; C24 at pad 51. Solder the ground pad (53). Configure both crystal load capacitors before use. Enable the internal DC/DC converter in firmware."
- note removed: "2.4GHz / PCB MIFA"
- note removed: "BMP581 / BMA400 / BMM350"
- note removed: "BUTTONS — ACTIVE LOW"
- note removed: "C22 at A3/A4/A9; C23 at G10; C24 at H1. Place regulator bypass at the corresponding balls."
- note removed: "Configure HF/LF internal load caps before starting crystals. Keep crystal traces short and clear of DCC / USB."
- note removed: "DEBUG — CORTEX SWD"
- note removed: "Enable VREGMAIN DC/DC in firmware."
- note removed: "LCD: R0=P2.00, R1=P2.04, G0=P2.06, G1=P2.08 B0=P2.09, B1=P2.10, BCK=P2.07. P2.00/P2.04 share SD DAT3/DAT1; FLPR arbitrates."
- note removed: "LS021B7DD02 display"
- note removed: "MAX-F11N L1/L5 GNSS"
- note removed: "Native 4-bit microSD"
- note removed: "PIEZO — 4kHz"
- note removed: "POWER PROBE PADS"
- note removed: "PREV/NEXT/BACK: GPIO pull-ups; firmware debounce. SELECT: PMIC_INT + SHPHLDSTATUS; enable SHPHLD events. Hold SELECT 10s: hardware power cycle (PMIC default)."
- note removed: "PWM21 CH0/CH1: antiphase, 4kHz, 50%; 6.4Vpp. H0H1 drive; hold both pins low when silent. Keep acoustic port clear; verify enclosed audibility."
- note removed: "R9: place at U6; tune from CLK waveform."
- note removed: "TC2030-CTX-NL: bare pads; no solder paste. VTref = +3V2 sense only. SWO unused; RTT over SWD. Keep probe access and alignment holes clear."
- note removed: "nRF54LM20A — SYSTEM / RF / USB"
- title: OpenBikeComputer — main board -> OpenBikeComputer - QFN main board
- moved on the sheet: C11, C12, C13, C21, C22, C23, C24, C25, C26, L3, L4, L6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
