File: hardware/projects/OBC_PCB/OBC_PCB.kicad_sch (KiCad schematic)
At the start: 22 parts, among them U6 nRF54LM20A-QGAA, Y1 32MHz, Y3 32.768kHz

Commit message: hardware: tidy the QFN schematic layout and style
Layout pass on the eight sheets. ERC stays at 0 violations on OBC_PCB and
USB_Baseboard. A netlist comparison shows the same 127 net partitions and
the same components, values and footprints.

Root sheet
- Draw SCL, SDA, COM_EN, LOUD, SHPHLD, BTN_SELECT and BUZZER_PWM as label
  stubs. Wire crossings fall from 38 to 0.
- Redraw the DCC/DECD/DECA/DECRF network as a chain without crossings.
- Move R5 and C26 clear of the crystal wires. Use a ground symbol on Y1
  instead of a label named GND.
- Hang the I2C test points on the U6C stubs.

Power sheet
- Attach the VBUS, VBAT and GND power flags to their nets.
- Tap TP1 onto the SHPHLD wire.
- Use a +3V2 symbol on LSIN2 instead of a label.
- Route SW2, the VSET straps and the CFG resistors without crossings.
- Move the SEL ground away from the LX1 pin.
- Show LSOUT1(GND) and INT(GND) for the unused LS1 and BMP581 pins.

Display, GNSS, user I/O
- Move J1 pin VA below VB so the VCOM/VB link no longer crosses VA.
- Move the GNSS FTE labels clear of the antenna pin 3 wire.
- Straighten the piezo wiring. Put the GND probe pad above its ground
  symbol.

Style
- One heading size (1.8 bold), one sub-heading size (1.27 bold) and one
  note size (1.0).
- Hide the voltage, dielectric and tolerance fields on the GNSS and radio
  sheets. Remove their dashed frames. Move both sheets to the top-left.
- Use Rev QFN and the same title format on every sheet.
- Set TP1 and TP2 to in_bom no like the other probe pads.
- Add C21 to the VDD bypass note.

Net names change for five nets because their labels are now on the root
sheet: BTN_SELECT, BUZZER_PWM, COM_EN, LOUD and SHPHLD. No net class
pattern uses them.

Co-Authored-By: Claude Sonnet 5.5 <noreply@anthropic.com>
Connections:
- net User I/O/BTN_SELECT renamed BTN_SELECT
- net User I/O/BUZZER_PWM renamed BUZZER_PWM
Other:
- note added: "VDD bypass: C22 at pad 6; C21 and C23 at pad 42; C24 at pad 51. Solder the ground pad (53). Configure both crystal load capacitors before use. Enable the internal DC/DC converter in firmware."
- note removed: "VDD bypass: C22 at pad 6; C23 at pad 42; C24 at pad 51. Solder the ground pad (53). Configure both crystal load capacitors before use. Enable the internal DC/DC converter in firmware."
- title: OpenBikeComputer - QFN main board -> OpenBikeComputer - main board
- moved on the sheet: C12, C13, C25, C26, L3, L4, L6, R5, TP11, TP12

Commit message: hardware: filter nRESET and add VCOM and VA probe pads
nRESET (pad 33) sits next to ANT (pad 34). Add a 1 kohm series resistor
(R68) and a 3.9 pF C0G capacitor to GND (C55) at the pad, as in Nordic's
nRF54L15 QFN48 reference circuit. The CSP98 references leave the pin
open, so they have no filter.

Add probe pads TP14 (VCOM) and TP15 (VA) on the display sheet for the
COM edge check at J1.

ERC stays at 0 violations. The netlist gains R68, C55, TP14 and TP15.
nRESET splits into the pad net and the external net.

Co-Authored-By: Claude Sonnet 5.5 <noreply@anthropic.com>
Parts:
- added C55: 3.9p, obc:C_Nordic_0201_0603Metric, symbol Device:C_Small
- added R68: 1k, Resistor_SMD:R_0201_0603Metric, symbol Device:R_Small
Connections:
- net GND: now also C55.2
- net nRESET: now also R68.2; no longer U6.33 (~{RESET})
- new net: C55.1, R68.1, U6.33 (~{RESET})
Other:
- note added: "VDD bypass: C22 at pad 6; C21 and C23 at pad 42; C24 at pad 51. R68 and C55 filter nRESET; place both at pad 33. Solder the ground pad (53). Configure both crystal load capacitors before use. Enable the internal DC/DC converter in firmware."
- note removed: "VDD bypass: C22 at pad 6; C21 and C23 at pad 42; C24 at pad 51. Solder the ground pad (53). Configure both crystal load capacitors before use. Enable the internal DC/DC converter in firmware."

Commit message: hardware: set the SD rail to 3.2 V, fix Y1 and tidy capacitor parts
- Power sheet note: BUCK1 runs at 3.2 V for the SD card, enabled after
  BUCK2 is at 3.2 V. C41 bias note follows. The +3V3_SD net keeps its
  name because the project net classes use it.
- Y1: CX2016DB32000D0FLJCC. It has +/-10 ppm tolerance and +/-15 ppm
  stability, 25 ppm in total against the 40 ppm Bluetooth LE limit in the
  nRF54LM20A HFXO specification. Same 2.0 x 1.6 mm package, 8 pF load.
- C47, C48 and C50 keep the dnp flag. Their value reads "tune (C0G)"
  instead of "DNP", so the BOM keeps the part class.
- C49 uses the same 2.2 uF 16 V X7R 0603 part as C39 and C40.

ERC stays at 0 violations. Only the three capacitor values change in the
netlist.

Co-Authored-By: Claude Sonnet 5.5 <noreply@anthropic.com>
Parts:
- Y1: Frequency tolerance 40ppm total -> 25ppm total; MPN CX2016DB32000D0WZRC1 -> CX2016DB32000D0FLJCC
Changed lines of the file:
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@@
 			)
 		)
-		(property "Description" "32MHz crystal, 8pF load, Nordic reference selection"
+		(property "Description" "32MHz crystal, 8pF load, +/-10ppm tolerance, +/-15ppm stability, -30 to 85C"
 			(at 360.68 69.85 0)
 			(hide yes)
@@
 			)
 		)
-		(property "Frequency tolerance" "40ppm total"
+		(property "Frequency tolerance" "25ppm total"
 			(at 129.54 0 0)
 			(hide yes)
@@
 			)
 		)
-		(property "MPN" "CX2016DB32000D0WZRC1"
+		(property "MPN" "CX2016DB32000D0FLJCC"
 			(at 129.54 0 0)
 			(hide yes)

Commit message: hardware: lay out the main sheet as a floor plan
Rebuild the root sheet around three aligned columns.

- Left: Power Management, Sensors, User I/O and GNSS. Right: Radio,
  Display and Storage. Centre: the four nRF54LM20A units in one stack,
  with a heading for the system block and each port.
- Every connection that can be a straight wire is a wire: USB, ANT, the
  LCD lines, the SD bus, buttons, buzzer, GNSS and ACC_INT1. SCL and SDA
  form a bus from Power Management to the sensors, port 1 and the display.
  COM_EN runs beside them. LOUD and SHPHLD run down the left margin.
- Labels remain only on PMIC_INT and on the SWD and reset nets. The debug
  header is on the far side of the page from the MCU.
- Name tags sit on the wires at the MCU pins, so each pin shows its
  function. They name the nets and connect nothing.
- Sheet names are module titles. Each sheet shows a one-line description.
- Two units get a new pin order in the symbol to match the floor plan:
  port 0 (buttons above GNSS) and P1.19 on port 1. Pad numbers and names
  are unchanged.
- The drawing is centred on the page. Wire crossings: two, where the I2C
  drops cross each other's bus.

ERC stays at 0 violations on both projects. Every net keeps the same
pins. Net names change for nine nets that now take their name from the
root sheet: ACC_INT1, BTN_PREV, BTN_NEXT, BTN_BACK, BTN_SELECT,
BUZZER_PWM, COM_EN, GPS_TXD and GPS_RXD. No net class pattern uses them.

Co-Authored-By: Claude Sonnet 5.5 <noreply@anthropic.com>
Connections:
- net GNSS/GPS_RXD renamed GPS_RXD
- net GNSS/GPS_TXD renamed GPS_TXD
- net Sensors/ACC_INT1 renamed ACC_INT1
- net User I/O/BTN_BACK renamed BTN_BACK
- net User I/O/BTN_NEXT renamed BTN_NEXT
- net User I/O/BTN_PREV renamed BTN_PREV
Other:
- note added: "2.4 GHz matching PCB MIFA antenna"
- note added: "4 buttons and piezo SWD header, reset"
- note added: "BMP581 pressure BMA400 motion wake LIS2MDL magnetometer"
- note added: "LS021B7DD02 panel electrode gates backlight driver"
- note added: "MAX-F11N L1/L5 GNSS"
- note added: "microSD card 4-bit sEMMC bus"
- note added: "nPM1300 PMIC and charger USB and battery input 3V2, SD and GNSS rails 5 V display supply"
- note added: "nRF54LM20A / PORT 0: BUTTONS, GNSS"
- note added: "nRF54LM20A / PORT 1: DISPLAY, I2C"
- note added: "nRF54LM20A / PORT 2: SD CARD"
- note added: "nRF54LM20A / SYSTEM, RF, USB"
- note removed: "MCU / CLOCKS / USB"
- moved on the sheet: C11, C12, C13, C21, C22, C23, C24, C25, C26, C55, L3, L4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
