File: hardware/projects/OBC_PCB/OBC_PCB.kicad_sch (KiCad schematic)
At the start: 24 parts, among them U6 nRF54LM20A-QGAA, Y1 32MHz, Y3 32.768kHz

Commit message: hardware: finalize shielded board placement and display flex integration
Parts:
- added R69, R70, R71, R72, R73, R74, R75: 100, Resistor_SMD:R_0201_0603Metric, symbol Device:R_Small
- added R76, R77, R78, R79, R80: 220, Resistor_SMD:R_0201_0603Metric, symbol Device:R_Small
- added SH1, SH2: BMI-S-202-F-20-R, obc:Laird_BMI-S-202-F-20_16.5mm, symbol obc:BMI-S-202-F-20-R
- added SH3, SH4: BMI-S-202-C-20, symbol obc:BMI-S-202-C-20
Connections:
- net BTN_PREV: now also U6.39 (P1.15); no longer U6.26 (P0.04)
- net BTN_SELECT: now also U6.26 (P0.04); no longer U6.39 (P1.15)
- net GND: now also SH1.1 (Shield), SH2.1 (Shield)
- net LCD_B0: now also R73.2; no longer U6.23 (P1.08)
- net LCD_B1: now also R74.2; no longer U6.24 (P1.09)
- net LCD_BCK: now also R75.2; no longer U6.15 (P1.05)
- net LCD_BSP: now also R80.2; no longer U6.41 (P1.18)
- net LCD_G0: now also R71.2; no longer U6.16 (P1.06)
- net LCD_G1: now also R72.2; no longer U6.22 (P1.07)
- net LCD_GCK: now also R76.2; no longer U6.40 (P1.16)
- net LCD_GEN: now also R78.2; no longer U6.12 (P1.02)
- net LCD_GSP: now also R77.2; no longer U6.11 (P1.01)
- net LCD_INTB: now also R79.2; no longer U6.50 (P1.24)
- net LCD_R0: now also R69.2; no longer U6.8 (P1.30)
- net LCD_R1: now also R70.2; no longer U6.9 (P1.31)
- net SCL: now also U6.41 (P1.18); no longer U6.13 (P1.03)
- net SDA: now also U6.40 (P1.16); no longer U6.14 (P1.04)
- new net LCD_B0_MCU: R73.1, U6.23 (P1.08)
- new net LCD_B1_MCU: R74.1, U6.24 (P1.09)
- new net LCD_BCK_MCU: R75.1, U6.15 (P1.05)
- new net LCD_BSP_MCU: R80.1, U6.13 (P1.03)
- new net LCD_G0_MCU: R71.1, U6.16 (P1.06)
- new net LCD_G1_MCU: R72.1, U6.22 (P1.07)
- new net LCD_GCK_MCU: R76.1, U6.14 (P1.04)
- new net LCD_GEN_MCU: R78.1, U6.12 (P1.02)
- new net LCD_GSP_MCU: R77.1, U6.11 (P1.01)
- new net LCD_INTB_MCU: R79.1, U6.50 (P1.24)
- new net LCD_R0_MCU: R69.1, U6.8 (P1.30)
- new net LCD_R1_MCU: R70.1, U6.9 (P1.31)
Other:
- note added: "EMI SHIELDS SH1 covers the MCU and clocks. Fit SH3. SH2 covers the PMIC and 5 V converter. Fit SH4. Both frames are BMI-S-202-F-20-R. Both removable lids are BMI-S-202-C-20. Bond frames to GND with a close via fence. Keep switching loops short and filter exits. Limit enclosed components to 1.8 mm height."
- note added: "LCD SOURCE DAMPING R69-R75: 100 Ohm, BCK and data. R76-R80: 220 Ohm, control. Place within 4 mm of U6. Use standard GPIO drive. Verify 10-90% edges at J1: target <=25 ns; panel limit 50 ns."
