File: hardware/projects/OBC_PCB/gnss.kicad_sch (KiCad schematic)
At the start: 14 parts, among them J8 RF coax pads, U1 MAX-F11N

Commit message: fix(hardware): apply schematic review and peripheral pin mapping
Parts:
- added C50: DNP, Capacitor_SMD:C_0402_1005Metric, symbol Device:C_Small
- ANT1: footprint obc:Taoglas_GGBLA125A_10x3.2mm_ContactPads -> obc:Taoglas_GGBLA125A_10x3.2mm_Corner
Connections:
- net GND: now also C50.2
- net at R40.1, U1.11 (RF_IN): now also C50.1

Commit message: hardware: name critical nets and ground connector tabs
Connections:
- net GNSS_RF_FEED: now reaches ANT1.1, C27.2, L7.1
- net GNSS_FTE1: now reaches ANT1.2 (FTE), R26.1
- net GNSS_FTE2: now reaches ANT1.3 (FTE), R27.1
- net GNSS_RF_IN: now reaches C50.1, R40.1, U1.11 (RF_IN)
- net GNSS_RF_TEST: now reaches C31.1, J8.1 (In), R40.2
- net GNSS_RF_MATCH: now reaches C27.1, C31.2, C32.1
Changed lines of the file:
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@@
 		(color 0 0 0 0)
 	)
+	(label "GNSS_RF_IN"
+		(at 134.62 97.79 0)
+		(effects
+			(font
+				(size 1 1)
+			)
+			(justify left bottom)
+		)
+	)
+	(label "GNSS_RF_TEST"
+		(at 152.4 104.14 0)
+		(effects
+			(font
+				(size 1 1)
+			)
+			(justify left bottom)
+		)
+	)
+	(label "GNSS_RF_MATCH"
+		(at 168.91 91.44 0)
+		(effects
+			(font
+				(size 1 1)
+			)
+			(justify left bottom)
+		)
+	)
+	(label "GNSS_RF_FEED"
+		(at 190.5 91.44 0)
+		(effects
+			(font
+				(size 1 1)
+			)
+			(justify left bottom)
+		)
+	)
+	(label "GNSS_FTE1"
+		(at 195.58 76.2 90)
+		(effects
+			(font
+				(size 1 1)
+			)
+			(justify right bottom)
+		)
+	)
+	(label "GNSS_FTE2"
+		(at 203.2 76.2 90)
+		(effects
+			(font
+				(size 1 1)
+			)
+			(justify right bottom)
+		)
+	)
 )

Commit message: hardware: prepare QFN schematic for non-HDI boards
Other:
- note added: "Release both UART pins before LS2 is off; enable LS2 before UARTE30. Set LS2 soft start to 50mA; measure V_IO at 25-3500us/V. V_BCKP ramp >=25us/V. Verify the production F11N power budget."
- note removed: "UART high-Z while GPS rail is off. Enable after BUCK2 = 3.2V. Verify LS2 startup: receiver VCC inrush up to 100mA. Preliminary F11N: recheck production pinout and power budget."
- moved on the sheet: C50
Changed lines of the file:
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@@
 		)
 	)
-	(text "UART high-Z while GPS rail is off. Enable after BUCK2 = 3.2V.\nVerify LS2 startup: receiver VCC inrush up to 100mA.\nPreliminary F11N: recheck production pinout and power budget."
+	(text "Release both UART pins before LS2 is off; enable LS2 before UARTE30.\nSet LS2 soft start to 50mA; measure V_IO at 25-3500us/V.\nV_BCKP ramp >=25us/V. Verify the production F11N power budget."
 		(at 85.09 144.78 0)
 		(effects
@@
 	(symbol
 		(lib_id "Device:C_Small")
-		(at 134.62 104.14 0)
+		(at 139.7 104.14 0)
 		(unit 1)
 		(body_style 1)
@@
 		(dnp yes)
 		(property "Reference" "C50"
-			(at 137.16 101.6 0)
+			(at 142.24 101.6 0)
 			(show_name no)
 			(do_not_autoplace no)
@@
 		)
 		(property "Value" "DNP"
-			(at 137.16 104.14 0)
+			(at 142.24 104.14 0)
 			(show_name no)
 			(do_not_autoplace no)
@@
 		)
 		(property "Footprint" "Capacitor_SMD:C_0402_1005Metric"
-			(at 134.62 104.14 0)
+			(at 139.7 104.14 0)
 			(hide yes)
 			(show_name no)
@@
 		)
 		(property "Datasheet" "https://www.taoglas.com/datasheets/GGBLA.125.A.pdf"
-			(at 134.62 104.14 0)
+			(at 139.7 104.14 0)
 			(hide yes)
 			(show_name no)
@@
 		)
 		(property "Description" "Optional RF input shunt capacitor; C0G, 25V, 0402; value set by RF measurement"
-			(at 134.62 104.14 0)
+			(at 139.7 104.14 0)
 			(hide yes)
 			(show_name no)
@@
 		)
 		(property "Manufacturer" "Murata"
-			(at -288.29 12.7 0)
+			(at -283.21 12.7 0)
 			(hide yes)
 			(effects
@@
 		)
 		(property "MPN" ""
-			(at -288.29 12.7 0)
+			(at -283.21 12.7 0)
 			(hide yes)
 			(effects
@@
 		)
 		(property "Voltage" "25V"
-			(at 137.16 106.68 0)
+			(at 142.24 106.68 0)
 			(effects
 				(font
@@
 		)
 		(property "Dielectric" "C0G"
-			(at 137.16 109.22 0)
+			(at 142.24 109.22 0)
 			(effects
 				(font
@@
 		)
 		(property "Tolerance" "0.1pF"
-			(at -288.29 12.7 0)
+			(at -283.21 12.7 0)
 			(hide yes)
 			(effects
@@
 		)
 		(property "Tuning" "Retune on final assembled PCB"
-			(at -288.29 12.7 0)
+			(at -283.21 12.7 0)
 			(hide yes)
 			(effects
@@
 	(symbol
 		(lib_id "power:GND")
-		(at 134.62 111.76 0)
+		(at 139.7 111.76 0)
 		(unit 1)
 		(body_style 1)
@@
 		(fields_autoplaced yes)
 		(property "Reference" "#PWR5001"
-			(at 137.16 107.95 0)
+			(at 142.24 107.95 0)
 			(hide yes)
 			(show_name no)
@@
 		)
 		(property "Value" "GND"
-			(at 137.16 109.22 0)
+			(at 142.24 109.22 0)
 			(hide yes)
 			(show_name no)
@@
 		)
 		(property "Footprint" ""
-			(at 137.16 110.49 0)
+			(at 142.24 110.49 0)
 			(hide yes)
 			(show_name no)
@@
 		)
 		(property "Datasheet" "~"
-			(at 137.16 111.76 0)
+			(at 142.24 111.76 0)
 			(hide yes)
 			(show_name no)
@@
 		)
 		(property "Description" ""
-			(at 137.16 113.03 0)
+			(at 142.24 113.03 0)
 			(hide yes)
 			(show_name no)
@@
 		(pts
 			(xy 132.08 91.44)
-			(xy 134.62 91.44)
-		)
-		(stroke
-			(width 0)
-			(type default)
-		)
-	)
-	(wire
-		(pts
-			(xy 134.62 91.44)
+			(xy 139.7 91.44)
+		)
+		(stroke
+			(width 0)
+			(type default)
+		)
+	)
+	(wire
+		(pts
+			(xy 139.7 91.44)
 			(xy 140.97 91.44)
 		)
@@
 	(wire
 		(pts
-			(xy 134.62 91.44)
-			(xy 134.62 101.6)
-		)
-		(stroke
-			(width 0)
-			(type default)
-		)
-	)
-	(wire
-		(pts
-			(xy 134.62 106.68)
-			(xy 134.62 111.76)
+			(xy 139.7 91.44)
+			(xy 139.7 101.6)
+		)
+		(stroke
+			(width 0)
+			(type default)
+		)
+	)
+	(wire
+		(pts
+			(xy 139.7 106.68)
+			(xy 139.7 111.76)
 		)
 		(stroke
@@
 	)
 	(junction
-		(at 134.62 91.44)
+		(at 139.7 91.44)
 		(diameter 0)
 		(color 0 0 0 0)
@@
 	)
 	(label "GNSS_RF_IN"
-		(at 134.62 97.79 0)
+		(at 139.7 97.79 0)
 		(effects
 			(font
@@
 	)
 	(label "GNSS_RF_MATCH"
-		(at 168.91 91.44 0)
+		(at 165.1 91.44 0)
 		(effects
 			(font
@@
 	)
 	(label "GNSS_FTE1"
-		(at 195.58 76.2 90)
+		(at 195.58 77.47 0)
 		(effects
 			(font
 				(size 1 1)
 			)
-			(justify right bottom)
+			(justify left bottom)
 		)
 	)
 	(label "GNSS_FTE2"
-		(at 203.2 76.2 90)
+		(at 205.74 77.47 0)
 		(effects
 			(font
 				(size 1 1)
 			)
-			(justify right bottom)
-		)
-	)
+			(justify left bottom)
+		)
+	)
