File: hardware/projects/OBC_PCB/gnss.kicad_sch (KiCad schematic)
At the start: 15 parts, among them J8 RF coax pads, U1 MAX-F11N

Commit message: hardware: finalize shielded board placement and display flex integration
Parts:
- C27: footprint Capacitor_SMD:C_0402_1005Metric -> Capacitor_SMD:C_0201_0603Metric; MPN GRM1555C1H100JA01D -> GJM0335C1E100JB01D; Voltage 50V -> 25V
- C31: footprint Capacitor_SMD:C_0402_1005Metric -> Capacitor_SMD:C_0201_0603Metric; MPN GRM1555C1H470JA01D -> GRM0335C1H470JA01D
- C32: footprint Capacitor_SMD:C_0402_1005Metric -> Capacitor_SMD:C_0201_0603Metric; MPN GJM1555C1H4R3BB01D -> GJM0335C1H4R3BB01D
Changed lines of the file:
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@@
 			)
 		)
-		(property "Footprint" "Capacitor_SMD:C_0402_1005Metric"
+		(property "Footprint" "Capacitor_SMD:C_0201_0603Metric"
 			(at 100.33 69.85 0)
 			(hide yes)
@@
 			)
 		)
-		(property "Datasheet" "https://www.taoglas.com/datasheets/GGBLA.125.A.pdf"
+		(property "Datasheet" "https://www.mouser.com/datasheet/2/281/1/GRM0335C1H470JA01_01A-1980894.pdf"
 			(at 100.33 71.12 0)
 			(hide yes)
@@
 			)
 		)
-		(property "MPN" "GRM1555C1H470JA01D"
+		(property "MPN" "GRM0335C1H470JA01D"
 			(at -317.5 -7.62 0)
 			(hide yes)
@@
 			)
 		)
-		(property "Footprint" "Capacitor_SMD:C_0402_1005Metric"
+		(property "Footprint" "Capacitor_SMD:C_0201_0603Metric"
 			(at 116.84 71.12 0)
 			(hide yes)
@@
 			)
 		)
-		(property "Datasheet" "https://www.taoglas.com/datasheets/GGBLA.125.A.pdf"
+		(property "Datasheet" "https://pim.murata.com/asset/pim4/ceramicCapacitorSMD/GJM0335C1E100JB01-31A-EN_PDF_CERAMICCAPACITORSMD"
 			(at 116.84 71.12 0)
 			(hide yes)
@@
 			)
 		)
-		(property "MPN" "GRM1555C1H100JA01D"
-			(at -317.5 -7.62 0)
-			(hide yes)
-			(effects
-				(font
-					(size 1.27 1.27)
-				)
-				(justify left)
-			)
-		)
-		(property "Voltage" "50V"
+		(property "MPN" "GJM0335C1E100JB01D"
+			(at -317.5 -7.62 0)
+			(hide yes)
+			(effects
+				(font
+					(size 1.27 1.27)
+				)
+				(justify left)
+			)
+		)
+		(property "Voltage" "25V"
 			(at 116.84 74.93 90)
 			(hide yes)
@@
 			)
 		)
-		(property "Footprint" "Capacitor_SMD:C_0402_1005Metric"
+		(property "Footprint" "Capacitor_SMD:C_0201_0603Metric"
 			(at 105.41 83.82 0)
 			(hide yes)
@@
 			)
 		)
-		(property "Datasheet" "https://www.taoglas.com/datasheets/GGBLA.125.A.pdf"
+		(property "Datasheet" "https://datasheet.octopart.com/GJM0335C1H4R3BB01D-Murata-datasheet-140568717.pdf"
 			(at 105.41 83.82 0)
 			(hide yes)
@@
 			)
 		)
-		(property "MPN" "GJM1555C1H4R3BB01D"
-			(at -317.5 -7.62 0)
-			(hide yes)
+		(property "MPN" "GJM0335C1H4R3BB01D"
+			(at -317.5 -7.62 0)
+			(hide yes)
