File: hardware/projects/OBC_PCB/gnss.kicad_sch (KiCad schematic)
At the start: 15 parts, among them J8 RF coax pads, U1 MAX-F11N

Commit message: hardware: add editable KiCad BOM and schematic exports
Parts:
- ANT1: Mouser (none) -> https://eu.mouser.com/en/ProductDetail/Taoglas/GGBLA.125.A?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; Price breaks EUR (none) -> 1:3.47;10:2.73;25:2.59;100:2.31;250:2.19;500:2.03;1000@1000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; Price checked (none) -> 2026-10-02; Price source (none) -> https://eu.mouser.com/en/ProductDetail/Taoglas/GGBLA.125.A?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; Sourcing notes (none) -> 645 in stock shown; further stock expected. 1000-piece reel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
- C27: DigiKey (none) -> https://www.digikey.de/en/products/detail/murata-electronic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; Mouser (none) -> https://www.mouser.com/ProductDetail/Murata-Electronics/GJM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; Price breaks EUR (none) -> 1:0.09;10:0.027;50:0.0184;100:0.0156;500:0.011; Price checked (none) -> 2026-10-02; Price source (none) -> https://www.digikey.de/en/products/detail/murata-electronic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
- C28: DigiKey (none) -> https://www.digikey.de/en/products/detail/samsung-electro-m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; MPN (none) -> CL05A225KP5NNNC; Manufacturer (none) -> Samsung Electro-Mechanics; Mouser (none) -> https://www.mouser.com/en/ProductDetail/Samsung-Electro-Mec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; Price breaks EUR (none) -> 1:0.12000;10:0.06700;50:0.04740;100:0.04110;500:0.03058;100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; Price checked (none) -> 2026-10-02; Price source (none) -> https://www.digikey.de/en/products/detail/samsung-electro-m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; Sourcing notes (none) -> Mouser shows limited stock; DigiKey EUR price used.
- C29, C30: DigiKey (none) -> https://www.digikey.de/en/products/detail/murata-electronic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; MPN (none) -> GRM155R71A104KA01D; Manufacturer (none) -> Murata; Price breaks EUR (none) -> 1:0.09000;10:0.02100;50:0.01400;100:0.01190;500:0.00830; Price checked (none) -> 2026-10-02; Price source (none) -> https://www.digikey.de/en/products/detail/murata-electronic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
- C31: Mouser (none) -> https://eu.mouser.com/en/ProductDetail/Murata-Electronics/G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; Price breaks EUR (none) -> 1:0.086;10:0.008;100:0.007;500:0.005;1000:0.004;2500:0.003; Price checked (none) -> 2026-10-02; Price source (none) -> https://eu.mouser.com/en/ProductDetail/Murata-Electronics/G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
- C32: Mouser (none) -> https://eu.mouser.com/ProductDetail/Murata-Electronics/GJM0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; Price breaks EUR (none) -> 1:0.086;10:0.04;50:0.028;100:0.024;500:0.017;4000:0.015;100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; Price checked (none) -> 2026-10-02; Price source (none) -> https://eu.mouser.com/ProductDetail/Murata-Electronics/GJM0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
- C50: Selection notes (none) -> DNP; choose value and MPN only after RF tuning.
- L7: DigiKey (none) -> https://www.digikey.de/en/products/detail/murata-electronic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; Mouser (none) -> https://www.mouser.com/en/ProductDetail/Murata-Electronics/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; Price breaks EUR (none) -> 1:0.10;10:0.082;100:0.0671;1000:0.05513;5000:0.04809; Price checked (none) -> 2026-10-02; Price source (none) -> https://www.digikey.de/en/products/detail/murata-electronic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
- R26, R27: Manufacturer Yageo -> YAGEO; Mouser (none) -> https://eu.mouser.com/en/ProductDetail/YAGEO/RC0402JR-070RL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; Power 63mW -> 62.5mW; Price breaks EUR (none) -> 1:0.086;10:0.005;100:0.003; Price checked (none) -> 2026-10-02; Price source (none) -> https://eu.mouser.com/en/ProductDetail/YAGEO/RC0402JR-070RL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; Rated Current (none) -> 1A; Resistance max (none) -> 50mOhm
- R40: MPN (none) -> RC0402JR-070RL; Manufacturer (none) -> YAGEO; Mouser (none) -> https://eu.mouser.com/en/ProductDetail/YAGEO/RC0402JR-070RL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; Power 63mW -> 62.5mW; Price breaks EUR (none) -> 1:0.086;10:0.005;100:0.003; Price checked (none) -> 2026-10-02; Price source (none) -> https://eu.mouser.com/en/ProductDetail/YAGEO/RC0402JR-070RL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; Rated Current (none) -> 1A; Resistance max (none) -> 50mOhm; Technology (none) -> Thick film; Voltage (none) -> 50V
- U1: Selection notes (none) -> No Mouser/DigiKey listing found; engineering samples pendin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; Sourcing notes (none) -> EUR unit-price tiers not verified; request quote.
