File: hardware/projects/OBC_PCB/display.kicad_sch (KiCad schematic)
At the start: 26 parts, among them J1 LS021B7DD02, J6 BACKLIGHT A/K - TBD, U8 SN74LVC02APWR, U9 LP5810BDSDR

Commit message: hardware: tidy the QFN schematic layout and style
Layout pass on the eight sheets. ERC stays at 0 violations on OBC_PCB and
USB_Baseboard. A netlist comparison shows the same 127 net partitions and
the same components, values and footprints.

Root sheet
- Draw SCL, SDA, COM_EN, LOUD, SHPHLD, BTN_SELECT and BUZZER_PWM as label
  stubs. Wire crossings fall from 38 to 0.
- Redraw the DCC/DECD/DECA/DECRF network as a chain without crossings.
- Move R5 and C26 clear of the crystal wires. Use a ground symbol on Y1
  instead of a label named GND.
- Hang the I2C test points on the U6C stubs.

Power sheet
- Attach the VBUS, VBAT and GND power flags to their nets.
- Tap TP1 onto the SHPHLD wire.
- Use a +3V2 symbol on LSIN2 instead of a label.
- Route SW2, the VSET straps and the CFG resistors without crossings.
- Move the SEL ground away from the LX1 pin.
- Show LSOUT1(GND) and INT(GND) for the unused LS1 and BMP581 pins.

Display, GNSS, user I/O
- Move J1 pin VA below VB so the VCOM/VB link no longer crosses VA.
- Move the GNSS FTE labels clear of the antenna pin 3 wire.
- Straighten the piezo wiring. Put the GND probe pad above its ground
  symbol.

Style
- One heading size (1.8 bold), one sub-heading size (1.27 bold) and one
  note size (1.0).
- Hide the voltage, dielectric and tolerance fields on the GNSS and radio
  sheets. Remove their dashed frames. Move both sheets to the top-left.
- Use Rev QFN and the same title format on every sheet.
- Set TP1 and TP2 to in_bom no like the other probe pads.
- Add C21 to the VDD bypass note.

Net names change for five nets because their labels are now on the root
sheet: BTN_SELECT, BUZZER_PWM, COM_EN, LOUD and SHPHLD. No net class
pattern uses them.

Co-Authored-By: Claude Sonnet 5.5 <noreply@anthropic.com>
Changed lines of the file:
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@@
 		(color 0 0 0 0)
 	)
-	(wire
-		(pts
-			(xy 172.72 71.12)
-			(xy 285.75 71.12)
-		)
-		(stroke
-			(width 0)
-			(type default)
-		)
-	)
-	(wire
-		(pts
-			(xy 285.75 71.12)
-			(xy 285.75 74.93)
-		)
-		(stroke
-			(width 0)
-			(type default)
-		)
-	)
-	(wire
-		(pts
-			(xy 285.75 74.93)
-			(xy 322.58 74.93)
-		)
-		(stroke
-			(width 0)
-			(type default)
-		)
-	)
 	(symbol
 		(lib_id "Device:C_Small")
@@
 		(effects
 			(font
-				(size 1.1 1.1)
+				(size 1.0 1.0)
 			)
 			(justify left top)
@@
 		(effects
 			(font
-				(size 1.05 1.05)
+				(size 1.0 1.0)
 			)
 			(justify left top)
@@
 		(effects
 			(font
-				(size 1 1)
+				(size 1.0 1.0)
 			)
 			(justify left top)
@@
 		(effects
 			(font
-				(size 1.5 1.5)
+				(size 1.8 1.8)
 				(bold yes)
 			)
@@
 		(effects
 			(font
-				(size 1.1 1.1)
+				(size 1.0 1.0)
 			)
 			(justify left top)
@@
 	)
 	(embedded_fonts no)
+	(wire
+		(pts
+			(xy 172.72 71.12)
+			(xy 260.35 71.12)
+		)
+		(stroke
+			(width 0)
+			(type default)
+		)
+	)
+	(wire
+		(pts
+			(xy 260.35 71.12)
+			(xy 260.35 80.01)
+		)
+		(stroke
+			(width 0)
+			(type default)
+		)
+	)
+	(wire
+		(pts
+			(xy 260.35 80.01)
+			(xy 322.58 80.01)
+		)
+		(stroke
+			(width 0)
+			(type default)
+		)
+	)
 )

Commit message: hardware: filter nRESET and add VCOM and VA probe pads
nRESET (pad 33) sits next to ANT (pad 34). Add a 1 kohm series resistor
(R68) and a 3.9 pF C0G capacitor to GND (C55) at the pad, as in Nordic's
nRF54L15 QFN48 reference circuit. The CSP98 references leave the pin
open, so they have no filter.

Add probe pads TP14 (VCOM) and TP15 (VA) on the display sheet for the
COM edge check at J1.

ERC stays at 0 violations. The netlist gains R68, C55, TP14 and TP15.
nRESET splits into the pad net and the external net.

Co-Authored-By: Claude Sonnet 5.5 <noreply@anthropic.com>
Parts:
- added TP14: VCOM, TestPoint:TestPoint_Pad_D1.0mm, symbol Connector:TestPoint
- added TP15: VA, TestPoint:TestPoint_Pad_D1.0mm, symbol Connector:TestPoint
Connections:
- net at J1.20 (VCOM), R48.2, R50.1: now also TP14.1
- net at J1.8 (VA), R49.2: now also TP15.1
Changed lines of the file:
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@@
 		)
 	)
+	(symbol
+		(lib_id "Connector:TestPoint")
+		(at 200.66 50.8 0)
+		(unit 1)
+		(exclude_from_sim no)
+		(in_bom no)
+		(on_board yes)
+		(dnp no)
+		(property "Footprint" "TestPoint:TestPoint_Pad_D1.0mm"
+			(at 0 0 0)
+			(hide yes)
+			(effects
+				(font
+					(size 1 1)
+				)
+				(justify left)
+			)
+		)
+		(property "Datasheet" ""
+			(at 0 0 0)
+			(hide yes)
+			(effects
+				(font
+					(size 1 1)
+				)
+				(justify left)
+			)
+		)
+		(property "Description" "Bare 1mm probe pad for VCOM; no fitted part or solder paste"
+			(at 0 0 0)
+			(hide yes)
+			(effects
+				(font
+					(size 1 1)
+				)
+				(justify left)
+			)
+		)
+		(property "Reference" "TP14"
+			(at 198.12 45.72 0)
+			(effects
+				(font
+					(size 1 1)
+				)
+				(justify right)
+			)
+		)
+		(property "Value" "VCOM"
+			(at 198.12 48.26 0)
+			(effects
+				(font
+					(size 1 1)
+				)
+				(justify right)
+			)
+		)
+		(instances
+			(project "OBC_PCB"
+				(path "/57e91c39-b072-457b-b097-52c5b44e61c8/6b8cca09-5e52-4203-8b94-2412467f33a4"
+					(reference "TP14")
+					(unit 1)
+				)
+			)
+		)
+		(pin "1"
+		)
+	)
+	(symbol
+		(lib_id "Connector:TestPoint")
+		(at 200.66 71.12 0)
+		(unit 1)
+		(exclude_from_sim no)
+		(in_bom no)
+		(on_board yes)
+		(dnp no)
+		(property "Footprint" "TestPoint:TestPoint_Pad_D1.0mm"
+			(at 0 0 0)
+			(hide yes)
+			(effects
+				(font
+					(size 1 1)
+				)
+				(justify left)
+			)
+		)
+		(property "Datasheet" ""
+			(at 0 0 0)
+			(hide yes)
+			(effects
+				(font
+					(size 1 1)
+				)
+				(justify left)
+			)
+		)
+		(property "Description" "Bare 1mm probe pad for VA; no fitted part or solder paste"
+			(at 0 0 0)
+			(hide yes)
+			(effects
+				(font
+					(size 1 1)
+				)
+				(justify left)
+			)
+		)
+		(property "Reference" "TP15"
+			(at 198.12 66.04 0)
+			(effects
+				(font
+					(size 1 1)
+				)
+				(justify right)
+			)
+		)
+		(property "Value" "VA"
+			(at 198.12 68.58 0)
+			(effects
+				(font
+					(size 1 1)
+				)
+				(justify right)
+			)
+		)
+		(instances
+			(project "OBC_PCB"
+				(path "/57e91c39-b072-457b-b097-52c5b44e61c8/6b8cca09-5e52-4203-8b94-2412467f33a4"
+					(reference "TP15")
+					(unit 1)
+				)
+			)
+		)
+		(pin "1"
+		)
+	)
+	(junction
+		(at 200.66 50.8)
+		(diameter 0)
+		(color 0 0 0 0)
+	)
+	(junction
+		(at 200.66 71.12)
+		(diameter 0)
+		(color 0 0 0 0)
+	)
 )

Commit message: hardware: set the SD rail to 3.2 V, fix Y1 and tidy capacitor parts
- Power sheet note: BUCK1 runs at 3.2 V for the SD card, enabled after
  BUCK2 is at 3.2 V. C41 bias note follows. The +3V3_SD net keeps its
  name because the project net classes use it.
- Y1: CX2016DB32000D0FLJCC. It has +/-10 ppm tolerance and +/-15 ppm
  stability, 25 ppm in total against the 40 ppm Bluetooth LE limit in the
  nRF54LM20A HFXO specification. Same 2.0 x 1.6 mm package, 8 pF load.
- C47, C48 and C50 keep the dnp flag. Their value reads "tune (C0G)"
  instead of "DNP", so the BOM keeps the part class.
- C49 uses the same 2.2 uF 16 V X7R 0603 part as C39 and C40.

ERC stays at 0 violations. Only the three capacitor values change in the
netlist.

Co-Authored-By: Claude Sonnet 5.5 <noreply@anthropic.com>
Parts:
- C49: Voltage 10V -> 16V
Changed lines of the file:
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@@
 			)
 		)
-		(property "Description" "2.2uF MLCC, 10V, X7R, 0603"
+		(property "Description" "Ceramic MLCC, 2.2uF, 16V, X7R, 10%, 0603"
 			(at 0 0 0)
 			(hide yes)
@@
 			)
 		)
-		(property "Voltage" "10V"
+		(property "Voltage" "16V"
 			(at 93.98 142.24 0)
 			(hide yes)

Commit message: hardware: consolidate capacitor parts
One part per value and footprint where the ratings allow it:

- 1 uF 0603 (C6, C14, C20, C44, C54): 25 V X7R, 10 %. Three ratings and
  two dielectrics become one part.
- 100 nF 0402 (17 parts): 10 V X7R, 10 %. C7, C16 and C17 move from X5R.
- 2.2 uF 0603: C15 joins C39, C40 and C49 at 16 V X7R.
- Descriptions, tolerances and ratings are now the same for every part of
  a value and footprint (2.2 uF 0402, 10 uF 0603, 10 uF 0805, generic
  descriptions on C51 to C54).

Four capacitor BOM lines fewer. The higher-rated X7R parts lose less
capacitance under DC bias than the X5R parts they replace. A 25 V 1 uF
0603 costs about 1 cent more than a 10 V one at 10 pieces.

ERC stays at 0 violations and the netlist is unchanged.

Co-Authored-By: Claude Sonnet 5.5 <noreply@anthropic.com>
Parts:
- C53: Tolerance (none) -> 10%
- C54: Tolerance (none) -> 10%; Voltage 10V -> 25V
Changed lines of the file:
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@@
 			)
 		)
-		(property "Description" "Unpolarized capacitor, small symbol"
+		(property "Description" "Ceramic MLCC, 100nF, 10V, X7R, 10%, 0402"
 			(at 0 0 0)
 			(hide yes)
@@
 				(font
 					(size 1 1)
+				)
+				(justify left)
+			)
+		)
+		(property "Tolerance" "10%"
+			(at 0 0 0)
+			(hide yes)
+			(effects
+				(font
+					(size 1.27 1.27)
 				)
 				(justify left)
@@
 			)
 		)
-		(property "Description" "Unpolarized capacitor, small symbol"
+		(property "Description" "Ceramic MLCC, 1uF, 25V, X7R, 10%, 0603"
 			(at 0 0 0)
 			(hide yes)
@@
 			)
 		)
-		(property "Voltage" "10V"
+		(property "Voltage" "25V"
 			(at 0 0 0)
 			(hide yes)
@@
 				)
 				(justify left)
+			)
+		)
+		(property "Tolerance" "10%"
+			(at 0 0 0)
+			(hide yes)
+			(effects
+				(font
+					(size 1.27 1.27)
+				)
+				(justify left)
