File: hardware/projects/OBC_PCB/display.kicad_sch (KiCad schematic)
At the start: 28 parts, among them J1 LS021B7DD02, J6 BACKLIGHT A/K - TBD, U8 SN74LVC02APWR, U9 LP5810BDSDR

Commit message: hardware: finalize shielded board placement and display flex integration
Parts:
- J1: symbol obc:LS021B7DD02 -> obc:LS021B7DD02_Underside; Pin Mapping (none) -> Underside fold: Molex pad n = Sharp pin 22-n; see Sharp rea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
- J6: value BACKLIGHT A/K - TBD -> BACKLIGHT A/K - PROVISIONAL SOLDER; footprint (none) -> obc:Backlight_Flex_Solder_2_P1.8mm_Provisional; Selection Status TBD: match backlight tail; do not fabricate connector footp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 -> PROVISIONAL: confirm tail width, pitch, polarity, LED topol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; now left out of the parts list
- U8: value SN74LVC02APWR -> SN74LVC02ABQAR; footprint Package_SO:TSSOP-14_4.4x5mm_P0.65mm -> Package_DFN_QFN:DHWQFN-14-1EP_2.5x3mm_P0.5mm_EP1x1.5mm; symbol obc:SN74LVC02APWR -> obc:SN74LVC02ABQAR; MPN SN74LVC02APWR -> SN74LVC02ABQAR
Connections:
- net +3V2: now also J1.13 (VDD1); no longer J1.9 (VDD1)
- net +5V_DISP: now also J1.21 (VDD2); no longer J1.1 (VDD2)
- net GND: now also J1.12 (VSS), U8.15 (EP); no longer J1.10 (VSS)
- net LCD_B0: now also J1.5 (B0); no longer J1.17 (B0)
- net LCD_B1: now also J1.4 (B1); no longer J1.18 (B1)
- net LCD_BCK: now also J1.10 (BCK); no longer J1.12 (BCK)
- net LCD_G0: now also J1.7 (G0); no longer J1.15 (G0)
- net LCD_G1: now also J1.6 (G1); no longer J1.16 (G1)
- net LCD_GCK: now also J1.18 (GCK); no longer J1.4 (GCK)
- net LCD_GEN: now also J1.17 (GEN); no longer J1.5 (GEN)
- net LCD_GSP: now also J1.19 (GSP); no longer J1.3 (GSP)
- net LCD_INTB: now also J1.16 (INTB); no longer J1.6 (INTB)
- net LCD_R0: now also J1.9 (R0); no longer J1.13 (R0)
- net LCD_R1: now also J1.8 (R1); no longer J1.14 (R1)
- net at R49.2, TP15.1: now also J1.14 (VA); no longer J1.8 (VA)
- net at R48.2, R50.1, TP14.1: now also J1.2 (VCOM); no longer J1.20 (VCOM)
- net at R50.2: now also J1.15 (VB); no longer J1.7 (VB)
Other:
- note added: "J1: underside fold reverses connector numbering. Molex pad n = Sharp LCD pin 22-n."
- note added: "J6 PROVISIONAL: 1.8 mm pitch, 1.2 x 3.0 mm solder pads. Confirm tail, polarity, LED load and solder/strain-relief process with supplier."
Changed lines of the file:
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@@
 	)
 	(symbol
-		(lib_id "obc:SN74LVC02APWR")
+		(lib_id "obc:SN74LVC02ABQAR")
 		(at 60.96 50.8 0)
 		(unit 1)
@@
 			)
 		)
-		(property "Value" "SN74LVC02APWR"
+		(property "Value" "SN74LVC02ABQAR"
 			(at 55.88 43.18 0)
 			(show_name no)
@@
 			)
 		)
-		(property "Footprint" "Package_SO:TSSOP-14_4.4x5mm_P0.65mm"
+		(property "Footprint" "Package_DFN_QFN:DHWQFN-14-1EP_2.5x3mm_P0.5mm_EP1x1.5mm"
 			(at 0 0 0)
 			(hide yes)
@@
 			)
 		)
-		(property "Description" "Quad 2-input NOR, 1.65-3.6V, TSSOP-14"
+		(property "Description" "Quad 2-input NOR, 1.65-3.6V, WQFN-14 with grounded exposed pad"
 			(at 0 0 0)
 			(hide yes)
@@
 			)
 		)
-		(property "MPN" "SN74LVC02APWR"
+		(property "MPN" "SN74LVC02ABQAR"
 			(at 0 0 0)
 			(hide yes)
@@
 	)
 	(symbol
-		(lib_id "obc:SN74LVC02APWR")
+		(lib_id "obc:SN74LVC02ABQAR")
 		(at 60.96 91.44 0)
 		(unit 2)
@@
 			)
 		)
-		(property "Value" "SN74LVC02APWR"
+		(property "Value" "SN74LVC02ABQAR"
 			(at 55.88 83.82 0)
 			(show_name no)
@@
 			)
 		)
-		(property "Footprint" "Package_SO:TSSOP-14_4.4x5mm_P0.65mm"
+		(property "Footprint" "Package_DFN_QFN:DHWQFN-14-1EP_2.5x3mm_P0.5mm_EP1x1.5mm"
 			(at 0 0 0)
 			(hide yes)
@@
 			)
 		)
-		(property "Description" "Quad 2-input NOR, 1.65-3.6V, TSSOP-14"
+		(property "Description" "Quad 2-input NOR, 1.65-3.6V, WQFN-14 with grounded exposed pad"
 			(at 0 0 0)
 			(hide yes)
@@
 			)
 		)
-		(property "MPN" "SN74LVC02APWR"
+		(property "MPN" "SN74LVC02ABQAR"
 			(at 0 0 0)
 			(hide yes)
@@
 	)
 	(symbol
-		(lib_id "obc:SN74LVC02APWR")
+		(lib_id "obc:SN74LVC02ABQAR")
 		(at 129.54 50.8 0)
 		(unit 3)
@@
 			)
 		)
-		(property "Value" "SN74LVC02APWR"
+		(property "Value" "SN74LVC02ABQAR"
 			(at 124.46 43.18 0)
 			(show_name no)
@@
 			)
 		)
-		(property "Footprint" "Package_SO:TSSOP-14_4.4x5mm_P0.65mm"
+		(property "Footprint" "Package_DFN_QFN:DHWQFN-14-1EP_2.5x3mm_P0.5mm_EP1x1.5mm"
 			(at 0 0 0)
 			(hide yes)
@@
 			)
 		)
-		(property "Description" "Quad 2-input NOR, 1.65-3.6V, TSSOP-14"
+		(property "Description" "Quad 2-input NOR, 1.65-3.6V, WQFN-14 with grounded exposed pad"
 			(at 0 0 0)
 			(hide yes)
@@
 			)
 		)
-		(property "MPN" "SN74LVC02APWR"
+		(property "MPN" "SN74LVC02ABQAR"
 			(at 0 0 0)
 			(hide yes)
@@
 	)
 	(symbol
-		(lib_id "obc:SN74LVC02APWR")
+		(lib_id "obc:SN74LVC02ABQAR")
 		(at 129.54 71.12 0)
 		(unit 4)
@@
 			)
 		)
-		(property "Value" "SN74LVC02APWR"
+		(property "Value" "SN74LVC02ABQAR"
 			(at 124.46 63.50000000000001 0)
 			(show_name no)
@@
 			)
 		)
-		(property "Footprint" "Package_SO:TSSOP-14_4.4x5mm_P0.65mm"
+		(property "Footprint" "Package_DFN_QFN:DHWQFN-14-1EP_2.5x3mm_P0.5mm_EP1x1.5mm"
 			(at 0 0 0)
 			(hide yes)
@@
 			)
 		)
-		(property "Description" "Quad 2-input NOR, 1.65-3.6V, TSSOP-14"
+		(property "Description" "Quad 2-input NOR, 1.65-3.6V, WQFN-14 with grounded exposed pad"
 			(at 0 0 0)
 			(hide yes)
@@
 			)
 		)
-		(property "MPN" "SN74LVC02APWR"
+		(property "MPN" "SN74LVC02ABQAR"
 			(at 0 0 0)
 			(hide yes)
@@
 	)
 	(symbol
-		(lib_id "obc:SN74LVC02APWR")
+		(lib_id "obc:SN74LVC02ABQAR")
 		(at 224.79 30.48 0)
 		(unit 5)
@@
 			)
 		)
-		(property "Value" "SN74LVC02APWR"
+		(property "Value" "SN74LVC02ABQAR"
 			(at 231.14 27.94 0)
 			(show_name no)
@@
 			)
 		)
-		(property "Footprint" "Package_SO:TSSOP-14_4.4x5mm_P0.65mm"
+		(property "Footprint" "Package_DFN_QFN:DHWQFN-14-1EP_2.5x3mm_P0.5mm_EP1x1.5mm"
 			(at 0.0 -5.08 0)
 			(hide yes)
@@
 			)
 		)
-		(property "Description" "Quad 2-input NOR, 1.65-3.6V, TSSOP-14"
+		(property "Description" "Quad 2-input NOR, 1.65-3.6V, WQFN-14 with grounded exposed pad"
 			(at 0.0 -5.08 0)
 			(hide yes)
@@
 			)
 		)
-		(property "MPN" "SN74LVC02APWR"
+		(property "MPN" "SN74LVC02ABQAR"
 			(at 0.0 -5.08 0)
 			(hide yes)
@@
 		(pin "14"
 		)
+		(pin "15"
+		)
 	)
 	(hierarchical_label "COM_SOURCE"
@@
 	)
 	(symbol
-		(lib_id "obc:LS021B7DD02")
+		(lib_id "obc:LS021B7DD02_Underside")
 		(at 342.9 91.44 0)
 		(unit 1)
@@
 			)
 		)
-		(property "Description" "FFC & FPC Connectors Easy-On .3mm FPC Conn RA BC 21Ckt"
+		(property "Description" "Sharp LS021B7DD02 with underside Molex 503566-2102: connector pad n mates LCD pin 22-n"
 			(at 178.816 129.032 0)
 			(hide yes)
@@
 			)
 		)
-		(pin "1"
+		(pin "21"
 		)
-		(pin "2"
+		(pin "20"
 		)
-		(pin "3"
+		(pin "19"
 		)
-		(pin "4"
+		(pin "18"
 		)
-		(pin "5"
+		(pin "17"
 		)
-		(pin "6"
+		(pin "16"
 		)
-		(pin "7"
+		(pin "15"
 		)
-		(pin "8"
+		(pin "14"
 		)
-		(pin "9"
+		(pin "13"
 		)
-		(pin "10"
+		(pin "12"
 		)
 		(pin "11"
 		)
-		(pin "12"
+		(pin "10"
 		)
-		(pin "13"
+		(pin "9"
 		)
-		(pin "14"
+		(pin "8"
 		)
-		(pin "15"
+		(pin "7"
 		)
-		(pin "16"
+		(pin "6"
 		)
-		(pin "17"
+		(pin "5"
 		)
-		(pin "18"
+		(pin "4"
 		)
-		(pin "19"
+		(pin "3"
 		)
-		(pin "20"
+		(pin "2"
 		)
-		(pin "21"
+		(pin "1"
 		)
 		(pin "MP1"
@@
 		(pin "MP2"
 		)
+		(property "Pin Mapping" "Underside fold: Molex pad n = Sharp pin 22-n; see Sharp rear contact-side outline"
+			(at 0 0 0)
+			(hide yes)
+			(effects
+				(font
+					(size 1.27 1.27)
+				)
+				(justify left)
+			)
+		)
 	)
 	(wire
@@
 		(unit 1)
 		(exclude_from_sim no)
-		(in_bom yes)
+		(in_bom no)
 		(on_board yes)
 		(dnp no)
-		(property "Footprint" ""
+		(property "Footprint" "obc:Backlight_Flex_Solder_2_P1.8mm_Provisional"
 			(at 0 0 0)
 			(hide yes)
@@
 			)
 		)
-		(property "Description" "Backlight connector; tail, pinout, LED topology and current not selected"
+		(property "Description" "Two direct-solder pads for custom backlight flex; 1=A (+5V_DISP), 2=K (BL_K); no connector fitted"
 			(at 0 0 0)
 			(hide yes)
@@
 			)
 		)
-		(property "Selection Status" "TBD: match backlight tail; do not fabricate connector footprint yet"
+		(property "Selection Status" "PROVISIONAL: confirm tail width, pitch, polarity, LED topology/current, solder process and strain relief with backlight manufacturer before fabrication"
 			(at 0 0 0)
 			(hide yes)
@@
 			)
 		)
-		(property "Value" "BACKLIGHT A/K - TBD"
+		(property "Value" "BACKLIGHT A/K - PROVISIONAL SOLDER"
 			(at 213.35999999999999 208.28 0)
 			(effects
@@
 		(color 0 0 0 0)
 	)
+	(wire
+		(pts
+			(xy 224.79 43.18)
+			(xy 227.33 43.18)
+		)
+		(stroke
+			(width 0)
+			(type default)
+		)
+	)
+	(text "J1: underside fold reverses connector numbering. Molex pad n = Sharp LCD pin 22-n."
+		(at 165.1 190.5 0)
+		(effects
+			(font
+				(size 1.27 1.27)
+			)
+			(justify left)
+		)
+	)
+	(text "J6 PROVISIONAL: 1.8 mm pitch, 1.2 x 3.0 mm solder pads. Confirm tail, polarity, LED load and solder/strain-relief process with supplier."
+		(at 165.1 233.68 0)
+		(effects
+			(font
+				(size 1.27 1.27)
+			)
+			(justify left)
+		)
+	)
 )

Commit message: hardware: add editable KiCad BOM and schematic exports
Parts:
- C39, C40, C49: DigiKey (none) -> https://www.digikey.com/en/products/detail/yageo/CC0603KRX7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; MPN (none) -> CC0603KRX7R7BB225; Manufacturer (none) -> YAGEO; Mouser (none) -> https://eu.mouser.com/de/ProductDetail/YAGEO/CC0603KRX7R7BB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; Price breaks EUR (none) -> 1:0.507;10:0.305;100:0.205;500:0.17;1000:0.158;2000:0.145; Price checked (none) -> 2026-10-02; Price source (none) -> https://eu.mouser.com/de/ProductDetail/YAGEO/CC0603KRX7R7BB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; Selection notes (none) -> Candidate; verify DC-bias, temperature and tolerance agains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
- C53: DigiKey (none) -> https://www.digikey.de/en/products/detail/murata-electronic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; MPN (none) -> GRM155R71A104KA01D; Manufacturer (none) -> Murata; Price breaks EUR (none) -> 1:0.09000;10:0.02100;50:0.01400;100:0.01190;500:0.00830; Price checked (none) -> 2026-10-02; Price source (none) -> https://www.digikey.de/en/products/detail/murata-electronic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
- C54: DigiKey (none) -> https://www.digikey.jp/ja/products/detail/yageo/CC0603KRX7R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; MPN (none) -> CC0603KRX7R8BB105; Manufacturer (none) -> YAGEO; Mouser (none) -> https://www.mouser.de/de/ProductDetail/YAGEO/CC0603KRX7R8BB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; Price breaks EUR (none) -> 1:0.215;10:0.108;100:0.08;500:0.065;1000:0.054; Price checked (none) -> 2026-10-02; Price source (none) -> https://www.mouser.de/de/ProductDetail/YAGEO/CC0603KRX7R8BB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
- J1: DigiKey (none) -> https://www.digikey.it/en/products/detail/molex/5035662102/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; Mouser (none) -> https://www.mouser.com/es/ProductDetail/Molex/503566-2102?q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; Sourcing notes (none) -> DigiKey lists factory minimum 48000; use Mouser cut tape fo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
- R46: MPN (none) -> RC0402FR-0747KL; Manufacturer (none) -> YAGEO; Mouser (none) -> https://eu.mouser.com/en/ProductDetail/YAGEO/RC0402FR-0747K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; Power (none) -> 62.5mW; Price breaks EUR (none) -> 1:0.086;10:0.009;100:0.006;1000:0.005;2500:0.003; Price checked (none) -> 2026-10-02; Price source (none) -> https://eu.mouser.com/en/ProductDetail/YAGEO/RC0402FR-0747K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; Technology (none) -> Thick film; Voltage (none) -> 50V
- R47, R51, R52, R53, R54, R55, R56, R57, R58, R59, R60, R61, R62: MPN (none) -> RC0402FR-07100KL; Manufacturer (none) -> YAGEO; Mouser (none) -> https://www.mouser.fr/en/ProductDetail/YAGEO/RC0402FR-07100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; Power (none) -> 62.5mW; Price breaks EUR (none) -> 1:0.086;10:0.009;100:0.006;1000:0.005;2500:0.003; Price checked (none) -> 2026-10-02; Price source (none) -> https://www.mouser.fr/en/ProductDetail/YAGEO/RC0402FR-07100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; Technology (none) -> Thick film; Voltage (none) -> 50V
- R48, R49: MPN (none) -> RC0402FR-07150RL; Manufacturer (none) -> YAGEO; Mouser (none) -> https://www.mouser.de/de/ProductDetail/YAGEO/RC0402FR-07150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; Power (none) -> 62.5mW; Price breaks EUR (none) -> 1:0.086;10:0.009;100:0.006;1000:0.005;2500:0.003; Price checked (none) -> 2026-10-02; Price source (none) -> https://www.mouser.de/de/ProductDetail/YAGEO/RC0402FR-07150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; Sourcing notes (none) -> Only 6 in stock shown; compare DigiKey before ordering.; Technology (none) -> Thick film; Voltage (none) -> 50V
- R50: MPN (none) -> RC0402JR-070RL; Manufacturer (none) -> YAGEO; Mouser (none) -> https://eu.mouser.com/en/ProductDetail/YAGEO/RC0402JR-070RL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; Power (none) -> 62.5mW; Price breaks EUR (none) -> 1:0.086;10:0.005;100:0.003; Price checked (none) -> 2026-10-02; Price source (none) -> https://eu.mouser.com/en/ProductDetail/YAGEO/RC0402JR-070RL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; Rated Current (none) -> 1A; Resistance max (none) -> 50mOhm; Technology (none) -> Thick film; Tolerance 1% -> Jumper; Voltage (none) -> 50V
- U8: Mouser (none) -> https://eu.mouser.com/en/ProductDetail/Texas-Instruments/SN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; Price breaks EUR (none) -> 1:0.378;10:0.263;25:0.235;100:0.204;250:0.188;500:0.18;1000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; Price checked (none) -> 2026-10-02; Price source (none) -> https://eu.mouser.com/en/ProductDetail/Texas-Instruments/SN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
- U9: DigiKey (none) -> https://www.digikey.de/en/products/detail/texas-instruments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; Mouser (none) -> https://eu.mouser.com/ProductDetail/Texas-Instruments/LP581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; Price breaks EUR (none) -> 1:0.74000;10:0.53100;25:0.47720;100:0.41930;250:0.39152;500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; Price checked (none) -> 2026-10-02; Price source (none) -> https://www.digikey.de/en/products/detail/texas-instruments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
