File: hardware/projects/OBC_PCB/sensors.kicad_sch (KiCad schematic)
At the start: 14 parts, among them U3 BMA400, U4 LIS2MDL, U5 BMP581

Commit message: hardware: tidy the QFN schematic layout and style
Layout pass on the eight sheets. ERC stays at 0 violations on OBC_PCB and
USB_Baseboard. A netlist comparison shows the same 127 net partitions and
the same components, values and footprints.

Root sheet
- Draw SCL, SDA, COM_EN, LOUD, SHPHLD, BTN_SELECT and BUZZER_PWM as label
  stubs. Wire crossings fall from 38 to 0.
- Redraw the DCC/DECD/DECA/DECRF network as a chain without crossings.
- Move R5 and C26 clear of the crystal wires. Use a ground symbol on Y1
  instead of a label named GND.
- Hang the I2C test points on the U6C stubs.

Power sheet
- Attach the VBUS, VBAT and GND power flags to their nets.
- Tap TP1 onto the SHPHLD wire.
- Use a +3V2 symbol on LSIN2 instead of a label.
- Route SW2, the VSET straps and the CFG resistors without crossings.
- Move the SEL ground away from the LX1 pin.
- Show LSOUT1(GND) and INT(GND) for the unused LS1 and BMP581 pins.

Display, GNSS, user I/O
- Move J1 pin VA below VB so the VCOM/VB link no longer crosses VA.
- Move the GNSS FTE labels clear of the antenna pin 3 wire.
- Straighten the piezo wiring. Put the GND probe pad above its ground
  symbol.

Style
- One heading size (1.8 bold), one sub-heading size (1.27 bold) and one
  note size (1.0).
- Hide the voltage, dielectric and tolerance fields on the GNSS and radio
  sheets. Remove their dashed frames. Move both sheets to the top-left.
- Use Rev QFN and the same title format on every sheet.
- Set TP1 and TP2 to in_bom no like the other probe pads.
- Add C21 to the VDD bypass note.

Net names change for five nets because their labels are now on the root
sheet: BTN_SELECT, BUZZER_PWM, COM_EN, LOUD and SHPHLD. No net class
pattern uses them.

Co-Authored-By: Claude Sonnet 5.5 <noreply@anthropic.com>
Changed lines of the file:
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@@
 		(effects
 			(font
-				(size 1.1 1.1)
+				(size 1.0 1.0)
 			)
 			(justify left top)
@@
 		(effects
 			(font
-				(size 1 1)
+				(size 1.0 1.0)
 			)
 			(justify left top)
@@
 		)
 		(pin "7"
-			(alternate "DISABLED")
+			(alternate "INT(GND)")
 		)
 		(pin "8"
@@
 		(effects
 			(font
-				(size 1.25 1.25)
+				(size 1.27 1.27)
 				(bold yes)
 			)
@@
 		(effects
 			(font
-				(size 1 1)
+				(size 1.0 1.0)
 			)
 			(justify left top)
@@
 		(effects
 			(font
-				(size 1.25 1.25)
+				(size 1.27 1.27)
 				(bold yes)
 			)
@@
 		(effects
 			(font
-				(size 1 1)
+				(size 1.0 1.0)
 			)
 			(justify left top)
@@
 		(effects
 			(font
-				(size 1.25 1.25)
+				(size 1.27 1.27)
 				(bold yes)
 			)
@@
 		(effects
 			(font
-				(size 1 1)
+				(size 1.0 1.0)
 			)
 			(justify left top)

Commit message: hardware: consolidate capacitor parts
One part per value and footprint where the ratings allow it:

- 1 uF 0603 (C6, C14, C20, C44, C54): 25 V X7R, 10 %. Three ratings and
  two dielectrics become one part.
- 100 nF 0402 (17 parts): 10 V X7R, 10 %. C7, C16 and C17 move from X5R.
- 2.2 uF 0603: C15 joins C39, C40 and C49 at 16 V X7R.
- Descriptions, tolerances and ratings are now the same for every part of
  a value and footprint (2.2 uF 0402, 10 uF 0603, 10 uF 0805, generic
  descriptions on C51 to C54).

Four capacitor BOM lines fewer. The higher-rated X7R parts lose less
capacitance under DC bias than the X5R parts they replace. A 25 V 1 uF
0603 costs about 1 cent more than a 10 V one at 10 pieces.

ERC stays at 0 violations and the netlist is unchanged.

Co-Authored-By: Claude Sonnet 5.5 <noreply@anthropic.com>
Parts:
- C51: Tolerance (none) -> 10%
Changed lines of the file:
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@@
 			)
 		)
-		(property "Description" "Unpolarized capacitor, small symbol"
+		(property "Description" "Ceramic MLCC, 10uF, 10V, X5R, 10%, 0603"
 			(at 0 0 0)
 			(hide yes)
@@
 				)
 				(justify left)
+			)
+		)
+		(property "Tolerance" "10%"
+			(at 0 0 0)
+			(hide yes)
+			(effects
+				(font
+					(size 1.27 1.27)
+				)
+				(justify left)
