File: hardware/projects/OBC_PCB/sensors.kicad_sch (KiCad schematic)
At the start: 14 parts, among them U3 BMA400, U4 LIS2MDL, U5 BMP581

Commit message: hardware: add editable KiCad BOM and schematic exports
Parts:
- C33, C34, C35, C36, C37, C38: DigiKey (none) -> https://www.digikey.de/en/products/detail/murata-electronic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; MPN (none) -> GRM155R71A104KA01D; Manufacturer (none) -> Murata; Price breaks EUR (none) -> 1:0.09000;10:0.02100;50:0.01400;100:0.01190;500:0.00830; Price checked (none) -> 2026-10-02; Price source (none) -> https://www.digikey.de/en/products/detail/murata-electronic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
- C42: MPN (none) -> GRM155R71A224KE01D; Manufacturer (none) -> Murata; Mouser (none) -> https://www.mouser.es/es/ProductDetail/Murata-Electronics/G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; Price breaks EUR (none) -> 1:0.086;10:0.024;100:0.021;500:0.015;1000:0.013;2500:0.011;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; Price checked (none) -> 2026-10-02; Price source (none) -> https://www.mouser.es/es/ProductDetail/Murata-Electronics/G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
- C51: MPN (none) -> C1608X5R1A106K080AC; Manufacturer (none) -> TDK; Mouser (none) -> https://eu.mouser.com/en/ProductDetail/TDK/C1608X5R1A106K08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; Price breaks EUR (none) -> 1:0.215;10:0.095;100:0.084;500:0.065;1000:0.058; Price checked (none) -> 2026-10-02; Price source (none) -> https://eu.mouser.com/en/ProductDetail/TDK/C1608X5R1A106K08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
- R23, R24: MPN (none) -> RC0402FR-074K7L; Manufacturer (none) -> YAGEO; Mouser (none) -> https://eu.mouser.com/en/ProductDetail/YAGEO/RC0402FR-074K7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; Power 63mW -> 62.5mW; Price breaks EUR (none) -> 1:0.086;10:0.008;100:0.006;1000:0.005;2500:0.003; Price checked (none) -> 2026-10-02; Price source (none) -> https://eu.mouser.com/en/ProductDetail/YAGEO/RC0402FR-074K7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
- R42: MPN (none) -> RC0402FR-07100KL; Manufacturer (none) -> YAGEO; Mouser (none) -> https://www.mouser.fr/en/ProductDetail/YAGEO/RC0402FR-07100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; Power (none) -> 62.5mW; Price breaks EUR (none) -> 1:0.086;10:0.009;100:0.006;1000:0.005;2500:0.003; Price checked (none) -> 2026-10-02; Price source (none) -> https://www.mouser.fr/en/ProductDetail/YAGEO/RC0402FR-07100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; Technology (none) -> Thick film; Voltage (none) -> 50V
- U3: Mouser (none) -> https://eu.mouser.com/ProductDetail/Bosch-Sensortec/BMA400?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; Price breaks EUR (none) -> 1:1.9;10:1.75;25:1.67;50:1.61;100:1.56;250:1.49;500:1.44;10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; Price checked (none) -> 2026-10-02; Price source (none) -> https://eu.mouser.com/ProductDetail/Bosch-Sensortec/BMA400?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
- U4: Mouser (none) -> https://eu.mouser.com/en/ProductDetail/STMicroelectronics/L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; Price breaks EUR (none) -> 1:2.37;5:2.11;10:1.90;50:1.77;100:1.67;500:1.49; Price checked (none) -> 2026-10-02; Price source (none) -> https://eu.mouser.com/en/ProductDetail/STMicroelectronics/L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; Sourcing notes (none) -> Backorder shown; confirm delivery and volume price.
- U5: Mouser (none) -> https://www.mouser.de/de/ProductDetail/Bosch-Sensortec/BMP5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; Price breaks EUR (none) -> 1:2.51;5:2.24;10:2.02;50:1.94;100:1.87;500:1.71;1000:1.66;2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; Price checked (none) -> 2026-10-02; Price source (none) -> https://www.mouser.de/de/ProductDetail/Bosch-Sensortec/BMP5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
