File: hardware/projects/OBC_PCB/radio.kicad_sch (KiCad schematic)
At the start: 11 parts, among them J7 RF coax pads

Commit message: hardware: add editable KiCad BOM and schematic exports
Parts:
- C45: DigiKey (none) -> https://www.digikey.fr/en/products/detail/murata-electronic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; Mouser (none) -> https://www.mouser.com/ProductDetail/Murata-Electronics/GJM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; Price breaks EUR (none) -> 1:0.11;10:0.06;50:0.0412;100:0.0358;500:0.02644; Price checked (none) -> 2026-10-02; Price source (none) -> https://www.digikey.fr/en/products/detail/murata-electronic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
- C46: DigiKey (none) -> https://www.digikey.de/de/products/detail/murata-electronic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; Mouser (none) -> https://www.mouser.com/en/ProductDetail/Murata-Electronics/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; Price breaks EUR (none) -> 1:0.10;10:0.052;50:0.0364;100:0.0315;500:0.02308; Price checked (none) -> 2026-10-02; Price source (none) -> https://www.digikey.de/de/products/detail/murata-electronic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
- C47, C48: Selection notes (none) -> DNP; choose value and MPN only after RF tuning.
- L10: DigiKey (none) -> https://www.digikey.de/en/products/detail/murata-electronic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; Mouser (none) -> https://www.mouser.com/es/ProductDetail/Murata-Electronics/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; Price breaks EUR (none) -> 1:0.11;10:0.092;100:0.0759;1000:0.06244;5000:0.05447; Price checked (none) -> 2026-10-02; Price source (none) -> https://www.digikey.de/en/products/detail/murata-electronic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; Selection notes (none) -> Provisional RF network; confirm QGAA matching with Nordic a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
- L8: DigiKey (none) -> https://www.digikey.fr/en/products/detail/murata-electronic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; Mouser (none) -> https://www.mouser.com/en/ProductDetail/Murata-Electronics/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; Price breaks EUR (none) -> 1:0.10;10:0.087;100:0.0717;1000:0.05891;5000:0.05138; Price checked (none) -> 2026-10-02; Price source (none) -> https://www.digikey.fr/en/products/detail/murata-electronic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; Selection notes (none) -> Provisional RF network; confirm QGAA matching with Nordic a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
- L9: DigiKey (none) -> https://www.digikey.es/en/products/detail/murata-electronic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; Mouser (none) -> https://www.mouser.com/es/ProductDetail/Murata-Electronics/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; Price breaks EUR (none) -> 1:0.10;10:0.087;100:0.0717;1000:0.05891;5000:0.05138; Price checked (none) -> 2026-10-02; Price source (none) -> https://www.digikey.es/en/products/detail/murata-electronic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; Selection notes (none) -> Provisional RF network; confirm QGAA matching with Nordic a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
- R35: MPN (none) -> RC0402JR-070RL; Manufacturer (none) -> YAGEO; Mouser (none) -> https://eu.mouser.com/en/ProductDetail/YAGEO/RC0402JR-070RL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; Power 63mW -> 62.5mW; Price breaks EUR (none) -> 1:0.086;10:0.005;100:0.003; Price checked (none) -> 2026-10-02; Price source (none) -> https://eu.mouser.com/en/ProductDetail/YAGEO/RC0402JR-070RL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; Rated Current (none) -> 1A; Resistance max (none) -> 50mOhm; Technology (none) -> Thick film; Tolerance (none) -> Jumper; Voltage (none) -> 50V
- R39: MPN (none) -> RC0402JR-070RL; Manufacturer (none) -> YAGEO; Mouser (none) -> https://eu.mouser.com/en/ProductDetail/YAGEO/RC0402JR-070RL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; Power 63mW -> 62.5mW; Price breaks EUR (none) -> 1:0.086;10:0.005;100:0.003; Price checked (none) -> 2026-10-02; Price source (none) -> https://eu.mouser.com/en/ProductDetail/YAGEO/RC0402JR-070RL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; Rated Current (none) -> 1A; Resistance max (none) -> 50mOhm; Technology (none) -> Thick film; Voltage (none) -> 50V
