File: hardware/projects/OBC_PCB/storage.kicad_sch (KiCad schematic)
At the start: 8 parts, among them J2 DM3CS-SF

Commit message: hardware: add editable KiCad BOM and schematic exports
Parts:
- C41: MPN (none) -> C1608X5R1A106K080AC; Manufacturer (none) -> TDK; Mouser (none) -> https://eu.mouser.com/en/ProductDetail/TDK/C1608X5R1A106K08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; Price breaks EUR (none) -> 1:0.215;10:0.095;100:0.084;500:0.065;1000:0.058; Price checked (none) -> 2026-10-02; Price source (none) -> https://eu.mouser.com/en/ProductDetail/TDK/C1608X5R1A106K08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; Selection notes (none) -> Candidate; verify DC-bias, temperature and tolerance agains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
- C43: DigiKey (none) -> https://www.digikey.de/en/products/detail/murata-electronic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; MPN (none) -> GRM155R71A104KA01D; Manufacturer (none) -> Murata; Price breaks EUR (none) -> 1:0.09000;10:0.02100;50:0.01400;100:0.01190;500:0.00830; Price checked (none) -> 2026-10-02; Price source (none) -> https://www.digikey.de/en/products/detail/murata-electronic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
- J2: Mouser (none) -> https://www.mouser.lu/fr/ProductDetail/Hirose-Connector/DM3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; Price breaks EUR (none) -> 1:1.72;10:1.47;25:1.31;100:1.25;250:1.12;500:1.06; Price checked (none) -> 2026-10-02; Price source (none) -> https://www.mouser.lu/fr/ProductDetail/Hirose-Connector/DM3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
- R28, R29, R30, R31, R32: MPN (none) -> RC0402FR-0747KL; Manufacturer (none) -> YAGEO; Mouser (none) -> https://eu.mouser.com/en/ProductDetail/YAGEO/RC0402FR-0747K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; Power 63mW -> 62.5mW; Price breaks EUR (none) -> 1:0.086;10:0.009;100:0.006;1000:0.005;2500:0.003; Price checked (none) -> 2026-10-02; Price source (none) -> https://eu.mouser.com/en/ProductDetail/YAGEO/RC0402FR-0747K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
