File: hardware/shared/power_management.kicad_sch (KiCad schematic)
At the start: 32 parts, among them J3 FH12-12S-0.5SH(55), J4 1S Li-Po, Q1 AO3400A, U2 nPM1300-QEAA, U7 TPS63900DSKR

Commit message: hardware: set the SD rail to 3.2 V, fix Y1 and tidy capacitor parts
- Power sheet note: BUCK1 runs at 3.2 V for the SD card, enabled after
  BUCK2 is at 3.2 V. C41 bias note follows. The +3V3_SD net keeps its
  name because the project net classes use it.
- Y1: CX2016DB32000D0FLJCC. It has +/-10 ppm tolerance and +/-15 ppm
  stability, 25 ppm in total against the 40 ppm Bluetooth LE limit in the
  nRF54LM20A HFXO specification. Same 2.0 x 1.6 mm package, 8 pF load.
- C47, C48 and C50 keep the dnp flag. Their value reads "tune (C0G)"
  instead of "DNP", so the BOM keeps the part class.
- C49 uses the same 2.2 uF 16 V X7R 0603 part as C39 and C40.

ERC stays at 0 violations. Only the three capacitor values change in the
netlist.

Co-Authored-By: Claude Sonnet 5.5 <noreply@anthropic.com>
Other:
- note added: "BUCK1: off at boot; set 3.2V for SD after BUCK2 is at 3.2V. BUCK2: 3.0V at boot; set 3.2V before LCD enable. LS1 unused: both pins grounded, keep disabled. LS2: +3V2_GPS; 50mA soft-start target."
- note removed: "BUCK1: off at boot; set 3.3V for SD. BUCK2: 3.0V at boot; set 3.2V before LCD enable. LS1 unused: both pins grounded, keep disabled. LS2: +3V2_GPS; 50mA soft-start target."
Changed lines of the file:
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@@
 		(color 0 0 0 0)
 	)
-	(text "BUCK1: off at boot; set 3.3V for SD.\nBUCK2: 3.0V at boot; set 3.2V before LCD enable.\nLS1 unused: both pins grounded, keep disabled.\nLS2: +3V2_GPS; 50mA soft-start target."
+	(text "BUCK1: off at boot; set 3.2V for SD after BUCK2 is at 3.2V.\nBUCK2: 3.0V at boot; set 3.2V before LCD enable.\nLS1 unused: both pins grounded, keep disabled.\nLS2: +3V2_GPS; 50mA soft-start target."
 		(at 198.12 137.16 0)
 		(effects

Commit message: hardware: consolidate capacitor parts
One part per value and footprint where the ratings allow it:

- 1 uF 0603 (C6, C14, C20, C44, C54): 25 V X7R, 10 %. Three ratings and
  two dielectrics become one part.
- 100 nF 0402 (17 parts): 10 V X7R, 10 %. C7, C16 and C17 move from X5R.
- 2.2 uF 0603: C15 joins C39, C40 and C49 at 16 V X7R.
- Descriptions, tolerances and ratings are now the same for every part of
  a value and footprint (2.2 uF 0402, 10 uF 0603, 10 uF 0805, generic
  descriptions on C51 to C54).

Four capacitor BOM lines fewer. The higher-rated X7R parts lose less
capacitance under DC bias than the X5R parts they replace. A 25 V 1 uF
0603 costs about 1 cent more than a 10 V one at 10 pieces.

ERC stays at 0 violations and the netlist is unchanged.

Co-Authored-By: Claude Sonnet 5.5 <noreply@anthropic.com>
Parts:
- C15: Dielectric X5R -> X7R; Voltage 10V -> 16V
- C16, C17, C7: Dielectric X5R -> X7R
- C20, C6: Dielectric X5R -> X7R; Voltage 10V -> 25V
Changed lines of the file:
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@@
 			)
 		)
-		(property "Description" "VBUS input MLCC, 1uF, 25V, X7R, 10%, 0603"
+		(property "Description" "Ceramic MLCC, 1uF, 25V, X7R, 10%, 0603"
 			(at 124.46 55.88 0)
 			(hide yes)
@@
 			)
 		)
-		(property "Description" "Ceramic MLCC, 10uF, 10V, X5R, 10%"
+		(property "Description" "Ceramic MLCC, 10uF, 10V, X5R, 10%, 0805"
 			(at 248.92 73.66 0)
 			(hide yes)
@@
 			)
 		)
-		(property "Description" "Ceramic MLCC, 100nF, 10V, X5R, 10%"
+		(property "Description" "Ceramic MLCC, 100nF, 10V, X7R, 10%, 0402"
 			(at 261.62 73.66 0)
 			(hide yes)
@@
 			)
 		)
-		(property "Dielectric" "X5R"
+		(property "Dielectric" "X7R"
 			(at 269.24 76.2 0)
 			(hide yes)
@@
 			)
 		)
-		(property "Description" "Ceramic MLCC, 10uF, 10V, X5R, 10%"
+		(property "Description" "Ceramic MLCC, 10uF, 10V, X5R, 10%, 0805"
 			(at 274.32 73.66 0)
 			(hide yes)
@@
 			)
 		)
-		(property "Description" "Ceramic MLCC, 10uF, 10V, X5R, 10%"
+		(property "Description" "Ceramic MLCC, 10uF, 10V, X5R, 10%, 0805"
 			(at 287.02 73.66 0)
 			(hide yes)
@@
 			)
 		)
-		(property "Description" "Ceramic MLCC, 100nF, 10V, X5R, 10%"
+		(property "Description" "Ceramic MLCC, 100nF, 10V, X7R, 10%, 0402"
 			(at 299.72 73.66 0)
 			(hide yes)
@@
 			)
 		)
-		(property "Dielectric" "X5R"
+		(property "Dielectric" "X7R"
 			(at 307.34 76.2 0)
 			(hide yes)
@@
 			)
 		)
-		(property "Description" "Ceramic MLCC, 100nF, 10V, X5R, 10%"
+		(property "Description" "Ceramic MLCC, 100nF, 10V, X7R, 10%, 0402"
 			(at 114.3 146.05 0)
 			(hide yes)
@@
 			)
 		)
-		(property "Dielectric" "X5R"
+		(property "Dielectric" "X7R"
 			(at 121.92 148.59 0)
 			(hide yes)
@@
 			)
 		)
-		(property "Description" "Ceramic MLCC, 1uF, 10V, X5R, 10%"
+		(property "Description" "Ceramic MLCC, 1uF, 25V, X7R, 10%, 0603"
 			(at 248.92 55.88 0)
 			(hide yes)
@@
 			)
 		)
-		(property "Voltage" "10V"
+		(property "Voltage" "25V"
 			(at 251.46 58.42 0)
 			(hide yes)
@@
 			)
 		)
-		(property "Dielectric" "X5R"
+		(property "Dielectric" "X7R"
 			(at 256.54 58.42 0)
 			(hide yes)
@@
 			)
 		)
-		(property "Description" "Ceramic MLCC, 10uF, 10V, X5R, 10%"
+		(property "Description" "Ceramic MLCC, 10uF, 10V, X5R, 10%, 0805"
 			(at 223.52 81.28 0)
 			(hide yes)
@@
 			)
 		)
-		(property "Description" "Ceramic MLCC, 10uF, 10V, X5R, 10%"
+		(property "Description" "Ceramic MLCC, 10uF, 10V, X5R, 10%, 0805"
 			(at 223.52 104.14 0)
 			(hide yes)
@@
 			)
 		)
-		(property "Description" "Ceramic MLCC, 1uF, 10V, X5R, 10%"
+		(property "Description" "Ceramic MLCC, 1uF, 25V, X7R, 10%, 0603"
 			(at 254.0 156.21 0)
 			(hide yes)
@@
 			)
 		)
-		(property "Voltage" "10V"
+		(property "Voltage" "25V"
 			(at 256.54 158.75 0)
 			(hide yes)
@@
 			)
 		)
-		(property "Dielectric" "X5R"
+		(property "Dielectric" "X7R"
 			(at 261.62 158.75 0)
 			(hide yes)
@@
 			)
 		)
-		(property "Description" "Ceramic MLCC, 2.2uF, 10V, X5R, 10%"
+		(property "Description" "Ceramic MLCC, 2.2uF, 16V, X7R, 10%, 0603"
 			(at 124.46 78.74 0)
 			(hide yes)
@@
 			)
 		)
-		(property "Voltage" "10V"
+		(property "Voltage" "16V"
 			(at 127.0 81.28 0)
 			(hide yes)
@@
 			)
 		)
-		(property "Dielectric" "X5R"
+		(property "Dielectric" "X7R"
 			(at 132.08 81.28 0)
 			(hide yes)
