File: hardware/shared/power_management.kicad_sch (KiCad schematic)
At the start: 32 parts, among them J3 FH12-12S-0.5SH(55), J4 1S Li-Po, Q1 AO3400A, U2 nPM1300-QEAA, U7 TPS63900DSKR

Commit message: hardware: finalize shielded board placement and display flex integration
Parts:
- J3: value FH12-12S-0.5SH(55) -> FH34SRJ-12S-0.5SH(50); footprint Connector_FFC-FPC:Hirose_FH12-12S-0.5SH_1x12-1MP_P0.50mm_Horizontal -> obc:Hirose_FH34SRJ_12S_0.5SH; Contact Side Bottom -> Top and bottom; gold contacts; FPC Thickness 0.30 +/-0.05mm -> 0.30 +/-0.03mm; MPN FH12-12S-0.5SH(55) -> FH34SRJ-12S-0.5SH(50)
- R64: footprint Resistor_SMD:R_0402_1005Metric -> Resistor_SMD:R_0201_0603Metric; MPN (none) -> RC0201FR-0710K5L; Manufacturer (none) -> Yageo
- R65: footprint Resistor_SMD:R_0402_1005Metric -> Resistor_SMD:R_0201_0603Metric; MPN (none) -> RC0201FR-0736K5L; Manufacturer (none) -> Yageo
Changed lines of the file:
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@@
 			)
 		)
-		(property "Value" "FH12-12S-0.5SH(55)"
+		(property "Value" "FH34SRJ-12S-0.5SH(50)"
 			(at 35.56 46.99 0)
 			(show_name no)
@@
 			)
 		)
-		(property "Footprint" "Connector_FFC-FPC:Hirose_FH12-12S-0.5SH_1x12-1MP_P0.50mm_Horizontal"
+		(property "Footprint" "obc:Hirose_FH34SRJ_12S_0.5SH"
 			(at 43.18 60.96 0)
 			(hide yes)
@@
 			)
 		)
-		(property "Datasheet" "https://www.hirose.com/en/product/p/CL0586-0704-0-55"
+		(property "Datasheet" "https://www.hirose.com/en/product/p/CL0580-1253-0-50"
 			(at 43.18 60.96 0)
 			(hide yes)
@@
 			)
 		)
-		(property "MPN" "FH12-12S-0.5SH(55)"
+		(property "MPN" "FH34SRJ-12S-0.5SH(50)"
 			(at 0 0 0)
 			(hide yes)
@@
 			)
 		)
-		(property "FPC Thickness" "0.30 +/-0.05mm"
+		(property "FPC Thickness" "0.30 +/-0.03mm"
 			(at 0 0 0)
 			(hide yes)
@@
 			)
 		)
-		(property "Contact Side" "Bottom"
+		(property "Contact Side" "Top and bottom; gold contacts"
 			(at 0 0 0)
 			(hide yes)
@@
 			)
 		)
-		(property "Footprint" "Resistor_SMD:R_0402_1005Metric"
+		(property "Footprint" "Resistor_SMD:R_0201_0603Metric"
 			(at 0 0 0)
 			(hide yes)
@@
 			)
 		)
-		(property "Datasheet" ""
+		(property "Datasheet" "https://yageogroup.com/content/datasheet/asset/file/PYU-RC_GROUP_51_ROHS_L"
 			(at 0 0 0)
 			(hide yes)
@@
 			)
 		)
-		(property "Description" "10.5k resistor, 1%, 0402"
+		(property "Description" "10.5k resistor, 1%, 0201"
 			(at 0 0 0)
 			(hide yes)
@@
 			)
 		)
-		(property "MPN" ""
+		(property "MPN" "RC0201FR-0710K5L"
 			(at 0 0 0)
 			(hide yes)
@@
 			)
 		)
-		(property "Manufacturer" ""
+		(property "Manufacturer" "Yageo"
 			(at 0 0 0)
 			(hide yes)
@@
 			)
 		)
-		(property "Footprint" "Resistor_SMD:R_0402_1005Metric"
+		(property "Footprint" "Resistor_SMD:R_0201_0603Metric"
 			(at -45.72 0 0)
 			(hide yes)
@@
 			)
 		)
-		(property "Datasheet" ""
+		(property "Datasheet" "https://yageogroup.com/content/datasheet/asset/file/PYU-RC_GROUP_51_ROHS_L"
 			(at -45.72 0 0)
 			(hide yes)
@@
 			)
 		)
-		(property "Description" "36.5k resistor, 1%, 0402"
+		(property "Description" "36.5k resistor, 1%, 0201"
 			(at -45.72 0 0)
 			(hide yes)
@@
 			)
 		)
-		(property "MPN" ""
+		(property "MPN" "RC0201FR-0736K5L"
 			(at -45.72 0 0)
 			(hide yes)
@@
 			)
 		)
-		(property "Manufacturer" ""
+		(property "Manufacturer" "Yageo"
 			(at -45.72 0 0)
 			(hide yes)

Commit message: hardware: consolidate USB baseboard, flex and connector assets
Bring the saved USB4730 baseboard, separate USB flex and battery metadata into the current shielded main-board branch. Preserve the main-board placement and circuit. Retain the existing connector assets. The saved FH12 flex tail still needs alignment with the main-board FH34SRJ connector before fabrication. Public docs unchanged.
Parts:
- J4: 3D model source (none) -> JST ACH catalogue; drawing-based model, not vendor CAD; Wire AWG28 for 2A rating -> AWG28; insulation OD 0.50-0.63 mm
Changed lines of the file:
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@@
 			)
 		)
-		(property "Description" "2-pin battery connector, 1.2mm pitch, 1.4mm mated height, 2A with AWG28"
+		(property "Description" "JST ACH, 2 contacts, 1.2 mm pitch, 1.4 mm mated height; 2 A with AWG28"
 			(at 40.64 120.65 0)
 			(hide yes)
@@
 			)
 		)
-		(property "Wire" "AWG28 for 2A rating"
+		(property "Wire" "AWG28; insulation OD 0.50-0.63 mm"
 			(at 0 0 0)
 			(hide yes)
@@
 			)
 		)
+		(property "3D model source" "JST ACH catalogue; drawing-based model, not vendor CAD"
+			(at 0 0 0)
+			(hide yes)
+			(effects
+				(font
+					(size 1.27 1.27)
+				)
+				(justify left)
+			)
+		)

Commit message: hardware: add editable KiCad BOM and schematic exports
Parts:
- C1, C2: MPN (none) -> C2012X5R1A106K085AC; Manufacturer (none) -> TDK; Mouser (none) -> https://eu.mouser.com/en/ProductDetail/TDK/C2012X5R1A106K08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; Price breaks EUR (none) -> 1:0.224;10:0.144;100:0.086;500:0.068;1000:0.062;2000:0.057; Price checked (none) -> 2026-10-02; Price source (none) -> https://eu.mouser.com/en/ProductDetail/TDK/C2012X5R1A106K08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; Selection notes (none) -> Candidate; verify total effective rail capacitance includin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
- C10, C9: MPN (none) -> C2012X5R1A226K125AB; Manufacturer (none) -> TDK; Mouser (none) -> https://eu.mouser.com/ProductDetail/TDK/C2012X5R1A226K125AB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; Price breaks EUR (none) -> 1:0.439;10:0.201;100:0.181;500:0.145;1000:0.135; Price checked (none) -> 2026-10-02; Price source (none) -> https://eu.mouser.com/ProductDetail/TDK/C2012X5R1A226K125AB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; Selection notes (none) -> Candidate; verify DC-bias, temperature and tolerance agains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
- C14, C20, C6: DigiKey (none) -> https://www.digikey.jp/ja/products/detail/yageo/CC0603KRX7R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; MPN (none) -> CC0603KRX7R8BB105; Manufacturer (none) -> YAGEO; Mouser (none) -> https://www.mouser.de/de/ProductDetail/YAGEO/CC0603KRX7R8BB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; Price breaks EUR (none) -> 1:0.215;10:0.108;100:0.08;500:0.065;1000:0.054; Price checked (none) -> 2026-10-02; Price source (none) -> https://www.mouser.de/de/ProductDetail/YAGEO/CC0603KRX7R8BB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
- C15: DigiKey (none) -> https://www.digikey.com/en/products/detail/yageo/CC0603KRX7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; MPN (none) -> CC0603KRX7R7BB225; Manufacturer (none) -> YAGEO; Mouser (none) -> https://eu.mouser.com/de/ProductDetail/YAGEO/CC0603KRX7R7BB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; Price breaks EUR (none) -> 1:0.507;10:0.305;100:0.205;500:0.17;1000:0.158;2000:0.145; Price checked (none) -> 2026-10-02; Price source (none) -> https://eu.mouser.com/de/ProductDetail/YAGEO/CC0603KRX7R7BB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
- C16, C17, C7: DigiKey (none) -> https://www.digikey.de/en/products/detail/murata-electronic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; MPN (none) -> GRM155R71A104KA01D; Manufacturer (none) -> Murata; Price breaks EUR (none) -> 1:0.09000;10:0.02100;50:0.01400;100:0.01190;500:0.00830; Price checked (none) -> 2026-10-02; Price source (none) -> https://www.digikey.de/en/products/detail/murata-electronic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
- C3, C4, C5, C8: MPN (none) -> C2012X5R1A106K085AC; Manufacturer (none) -> TDK; Mouser (none) -> https://eu.mouser.com/en/ProductDetail/TDK/C2012X5R1A106K08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; Price breaks EUR (none) -> 1:0.224;10:0.144;100:0.086;500:0.068;1000:0.062;2000:0.057; Price checked (none) -> 2026-10-02; Price source (none) -> https://eu.mouser.com/en/ProductDetail/TDK/C2012X5R1A106K08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; Selection notes (none) -> Candidate; verify DC-bias, temperature and tolerance agains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
- J3: DigiKey (none) -> https://www.digikey.gr/en/products/detail/hirose-electric-c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; Price breaks EUR (none) -> 1:1.00000;10:0.85300;25:0.79920;50:0.76100;100:0.72460;250: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; Price checked (none) -> 2026-10-02; Price source (none) -> https://www.digikey.gr/en/products/detail/hirose-electric-c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
- J4: Mouser (none) -> https://eu.mouser.com/en/ProductDetail/JST-Commercial/BM02B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; Price breaks EUR (none) -> 1:0.439;10:0.374;100:0.318;250:0.284;1000:0.27;2500:0.207; Price checked (none) -> 2026-10-02; Price source (none) -> https://eu.mouser.com/en/ProductDetail/JST-Commercial/BM02B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; Sourcing notes (none) -> Supplier lists the lead-free suffix (LF)(SN).
- L1, L2, L5: Mouser (none) -> https://www.mouser.lt/lt/ProductDetail/Wurth-Elektronik/744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; Price breaks EUR (none) -> 1:1.01;50:0.842;250:0.78;500:0.699; Price checked (none) -> 2026-10-02; Price source (none) -> https://www.mouser.lt/lt/ProductDetail/Wurth-Elektronik/744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
- Q1: DigiKey (none) -> https://www.digikey.de/en/products/detail/alpha-omega-semic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; Price breaks EUR (none) -> 1:0.45;10:0.276;50:0.1996;100:0.1749;500:0.13112; Price checked (none) -> 2026-10-02; Price source (none) -> https://www.digikey.de/en/products/detail/alpha-omega-semic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
- R1: MPN (none) -> RC0402JR-070RL; Manufacturer (none) -> YAGEO; Mouser (none) -> https://eu.mouser.com/en/ProductDetail/YAGEO/RC0402JR-070RL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; Power 63mW -> 62.5mW; Price breaks EUR (none) -> 1:0.086;10:0.005;100:0.003; Price checked (none) -> 2026-10-02; Price source (none) -> https://eu.mouser.com/en/ProductDetail/YAGEO/RC0402JR-070RL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; Rated Current (none) -> 1A; Resistance max (none) -> 50mOhm; Tolerance 1% -> Jumper
- R2: MPN (none) -> RC0402FR-07150KL; Manufacturer (none) -> YAGEO; Mouser (none) -> https://eu.mouser.com/de/ProductDetail/YAGEO/RC0402FR-07150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; Power 63mW -> 62.5mW; Price breaks EUR (none) -> 1:0.086;10:0.008;100:0.006;1000:0.005;2500:0.003; Price checked (none) -> 2026-10-02; Price source (none) -> https://eu.mouser.com/de/ProductDetail/YAGEO/RC0402FR-07150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
- R3: MPN (none) -> RC0402FR-071ML; Manufacturer (none) -> YAGEO; Mouser (none) -> https://eu.mouser.com/en/ProductDetail/YAGEO/RC0402FR-071ML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; Power 63mW -> 62.5mW; Price breaks EUR (none) -> 1:0.086;10:0.008;100:0.006;1000:0.005;2500:0.003; Price checked (none) -> 2026-10-02; Price source (none) -> https://eu.mouser.com/en/ProductDetail/YAGEO/RC0402FR-071ML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
- R63: MPN (none) -> RC0402FR-0736K5L; Manufacturer (none) -> YAGEO; Mouser (none) -> https://www.mouser.fr/fr/ProductDetail/YAGEO/RC0402FR-0736K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; Power (none) -> 62.5mW; Price breaks EUR (none) -> 1:0.086;10:0.009;100:0.005;2500:0.003; Price checked (none) -> 2026-10-02; Price source (none) -> https://www.mouser.fr/fr/ProductDetail/YAGEO/RC0402FR-0736K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; Technology (none) -> Thick film; Voltage (none) -> 50V
- R64: Manufacturer Yageo -> YAGEO; Mouser (none) -> https://www.mouser.es/ProductDetail/YAGEO/RC0201FR-0710K5L?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; Power (none) -> 50mW; Price breaks EUR (none) -> 1:0.086;10:0.009;100:0.007;1000:0.005; Price checked (none) -> 2026-10-02; Price source (none) -> https://www.mouser.es/ProductDetail/YAGEO/RC0201FR-0710K5L?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; Technology (none) -> Thick film; Voltage (none) -> 25V
- R65: Manufacturer Yageo -> YAGEO; Mouser (none) -> https://eu.mouser.com/pl/ProductDetail/YAGEO/RC0201FR-0736K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; Power (none) -> 50mW; Price breaks EUR (none) -> 1:0.146;10:0.015;100:0.01;1000:0.009; Price checked (none) -> 2026-10-02; Price source (none) -> https://eu.mouser.com/pl/ProductDetail/YAGEO/RC0201FR-0736K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; Technology (none) -> Thick film; Voltage (none) -> 25V
- R66: MPN (none) -> ERJ-2RKF1001X; Manufacturer (none) -> Panasonic; Mouser (none) -> https://eu.mouser.com/en/ProductDetail/Panasonic-Industry/E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; Power >=63mW -> 100mW; Price breaks EUR (none) -> 1:0.086;10:0.016;100:0.014;250:0.011;500:0.009;1000:0.008;5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; Price checked (none) -> 2026-10-02; Price source (none) -> https://eu.mouser.com/en/ProductDetail/Panasonic-Industry/E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; Technology (none) -> Thick film; Voltage (none) -> 50V
- R67: MPN (none) -> RC0402FR-07100KL; Manufacturer (none) -> YAGEO; Mouser (none) -> https://www.mouser.fr/en/ProductDetail/YAGEO/RC0402FR-07100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; Power (none) -> 62.5mW; Price breaks EUR (none) -> 1:0.086;10:0.009;100:0.006;1000:0.005;2500:0.003; Price checked (none) -> 2026-10-02; Price source (none) -> https://www.mouser.fr/en/ProductDetail/YAGEO/RC0402FR-07100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; Technology (none) -> Thick film; Voltage (none) -> 50V
- U2: Mouser (none) -> https://eu.mouser.com/tr/ProductDetail/Nordic-Semiconductor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; Price breaks EUR (none) -> 1:2.57;10:1.92;25:1.75;100:1.57;250:1.49;500:1.45;1000:1.38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; Price checked (none) -> 2026-10-02; Price source (none) -> https://eu.mouser.com/tr/ProductDetail/Nordic-Semiconductor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; Sourcing notes (none) -> Backorder shown; confirm delivery.
- U7: DigiKey (none) -> https://www.digikey.fr/en/products/detail/texas-instruments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; Mouser (none) -> https://www.mouser.fr/en/ProductDetail/Texas-Instruments/TP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; Price breaks EUR (none) -> 1:2.36;10:1.75;25:1.6;100:1.44;250:1.36;500:1.32;1000:1.26; Price checked (none) -> 2026-10-02; Price source (none) -> https://www.mouser.fr/en/ProductDetail/Texas-Instruments/TP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; Sourcing notes (none) -> Limited Mouser stock shown; DigiKey has more stock.
